File: TUSB4041I_4-port_USB20_hub.kicad_sch (KiCad schematic)
At the start: 22 parts, among them U1001 TUSB4041I

Commit message: Major update, everything has been touched
Parts:
- R410: renamed from R1009; footprint (none) -> cubesat_rp2040:R_0402_1005Metric
- renumbered C1013 to C413, C1012 to C414, C1005 to C415, C1006 to C416, C1007 to C417, C1008 to C418, C1009 to C419, C1010 to C420, C1011 to C421, C1001 to C422, C1002 to C423, C1003 to C424, C1004 to C425, R1001 to R408, R1002 to R409, R1004 to R411, R1005 to R412, R1006 to R413, R1007 to R414, R1008 to R415, U1001 to U402
