File: cubesat_bus.kicad_sch (KiCad schematic)
At the start: 2 parts

Commit message: Block diagram
Parts:
- H1, H2: footprint cubesat_rp2040:SAMTEC_ESQ-126-39-G-D -> cubesat_rp2040:ESQ-126-Y-X-D
Changed lines of the file:
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@@
 			)
 		)
-		(property "Footprint" "cubesat_rp2040:SAMTEC_ESQ-126-39-G-D"
+		(property "Footprint" "cubesat_rp2040:ESQ-126-Y-X-D"
 			(at 161.29 67.31 0)
 			(effects
@@
 			)
 		)
-		(property "Footprint" "cubesat_rp2040:SAMTEC_ESQ-126-39-G-D"
+		(property "Footprint" "cubesat_rp2040:ESQ-126-Y-X-D"
 			(at 110.49 67.31 0)
 			(effects

Commit message: Update footprints, route more circuit blocks
Parts:
- H1, H2: footprint cubesat_rp2040:ESQ-126-Y-X-D -> cubesat_rp2040:SAMTEC_ESQ-126-39-G-D
Changed lines of the file:
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@@
 			)
 		)
-		(property "Footprint" "cubesat_rp2040:ESQ-126-Y-X-D"
+		(property "Footprint" "cubesat_rp2040:SAMTEC_ESQ-126-39-G-D"
 			(at 161.29 67.31 0)
 			(effects
@@
 			)
 		)
-		(property "Footprint" "cubesat_rp2040:ESQ-126-Y-X-D"
+		(property "Footprint" "cubesat_rp2040:SAMTEC_ESQ-126-39-G-D"
 			(at 110.49 67.31 0)
 			(effects

Commit message: Big update, bad commit messsage :)
Parts:
- renumbered H1 to H601, H2 to H602
Other:
- company: (none) -> Magnus Oksbøl Therkelsen
- title: (none) -> CubeSat RP2040 Board
Changed lines of the file:
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@@
 	(generator_version "8.0")
 	(paper "A4")
+	(title_block
+		(title "CubeSat RP2040 Board")
+		(rev "1")
+		(company "Magnus Oksbøl Therkelsen")
+		(comment 1 "Author: Magnus Oksbøl Therkelsen")
+		(comment 2 "Checked by: ")
+	)
 	(no_connect
 		(at 97.79 67.31)
@@
 		(dnp no)
 		(fields_autoplaced yes)
-		(property "Reference" "H2"
+		(property "Reference" "H602"
 			(at 161.29 26.67 0)
 			(effects
@@
 			(project "cubesat_rp2040"
 				(path "/5511013b-c214-40ba-8960-f470f52474f8/0c29b30e-7660-45bf-be81-5710013bc73b"
-					(reference "H2")
+					(reference "H602")
 					(unit 1)
 				)
@@
 		(dnp no)
 		(fields_autoplaced yes)
-		(property "Reference" "H1"
+		(property "Reference" "H601"
 			(at 110.49 26.67 0)
 			(effects
@@
 			(project "cubesat_rp2040"
 				(path "/5511013b-c214-40ba-8960-f470f52474f8/0c29b30e-7660-45bf-be81-5710013bc73b"
-					(reference "H1")
+					(reference "H601")
 					(unit 1)
 				)

Commit message: Major update, everything has been touched
Parts:
- renumbered H601 to H501, H602 to H502
Changed lines of the file:
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@@
 	(generator "eeschema")
 	(generator_version "8.0")
-	(paper "A4")
+	(paper "A3")
 	(title_block
 		(title "CubeSat RP2040 Board")
@@
 		(dnp no)
 		(fields_autoplaced yes)
-		(property "Reference" "H602"
+		(property "Reference" "H502"
 			(at 161.29 26.67 0)
 			(effects
@@
 			(project "cubesat_rp2040"
 				(path "/5511013b-c214-40ba-8960-f470f52474f8/0c29b30e-7660-45bf-be81-5710013bc73b"
-					(reference "H602")
+					(reference "H502")
 					(unit 1)
 				)
@@
 		(dnp no)
 		(fields_autoplaced yes)
-		(property "Reference" "H601"
+		(property "Reference" "H501"
 			(at 110.49 26.67 0)
 			(effects
@@
 			(project "cubesat_rp2040"
 				(path "/5511013b-c214-40ba-8960-f470f52474f8/0c29b30e-7660-45bf-be81-5710013bc73b"
-					(reference "H601")
+					(reference "H501")
 					(unit 1)
 				)
