File: cubesat_rp2040.kicad_pcb (KiCad board)
At the start: 4 copper layers, 90.2 x 95.9 mm, 89 parts, among them J101 Conn_01x02, J102 ESQ-126-39-G-D, J103 ESQ-126-39-G-D, J301 USB_C_Receptacle_USB2.0, J501 FTSH-105-01-L-DV-007, SW101 SW_Push, U201 L7983, U301 TUSB4041I, U401 T6405 R24M0, U502 RP2040, U503 S25FL128SAGNFM000

Commit message: Another large revision, but we are getting closer
Parts:
- removed H101, H102, H103, H104: MountingHole_Pad, MountingHole:MountingHole_3.2mm_M3_Pad_Via
- removed J101: Conn_01x02, Connector_PinHeader_2.54mm:PinHeader_1x02_P2.54mm_Horizontal
- removed J102, J103: ESQ-126-39-G-D, cubesat_rp2040:SAMTEC_ESQ-126-39-G-D
- removed R501, R502: 0R, cubesat_rp2040:R_0402_1005Metric
- removed R507: 100k, cubesat_rp2040:R_0402_1005Metric
- removed U401: T6405 R24M0, cubesat_rp2040:Crystal_SMD_Rakon_3225-4Pin_3.2x2.5mm
- removed kibuzzard-66B1EB87: G***, kibuzzard-66B1EB87
- removed kibuzzard-66B1EBBE: G***, kibuzzard-66B1EBBE
- removed kibuzzard-66B4F7EF: G***, kibuzzard-66B4F7EF
- added C23: 15pF, cubesat_rp2040:C_0402_1005Metric, B.Cu at (118.6, 105.8)
- added C25: 10uF, Capacitor_SMD:C_1206_3216Metric, F.Cu at (11.3, 150.5)
- added C26: 100nF, cubesat_rp2040:C_0402_1005Metric, F.Cu at (15.6, 149.8)
- added C27: 1uF, Capacitor_SMD:C_0805_2012Metric, F.Cu at (10.8, 157.0)
- added C28: 100nF, cubesat_rp2040:C_0402_1005Metric, F.Cu at (15.6, 151.8)
- added C29: 10uF, Capacitor_SMD:C_1206_3216Metric, F.Cu at (11.3, 153.8)
- added C30: 100nF, cubesat_rp2040:C_0402_1005Metric, F.Cu at (-1.79, 198.1)
- added C45: 100nF, cubesat_rp2040:C_0402_1005Metric, F.Cu at (62.5, 65.2)
- added C46: 100nF, cubesat_rp2040:C_0402_1005Metric, F.Cu at (68.7, 65.9)
- added C47: 4.7nF, cubesat_rp2040:C_0402_1005Metric, F.Cu at (68.7, 62.9)
- added C48: 4.7nF, cubesat_rp2040:C_0402_1005Metric, F.Cu at (68.7, 68.9)
- added C49: 100nF, cubesat_rp2040:C_0402_1005Metric, F.Cu at (30.3, 180.8)
- added C50: 10uF, Capacitor_SMD:C_1206_3216Metric, F.Cu at (0.83, 162.2)
- added C51: 100nF, cubesat_rp2040:C_0402_1005Metric, F.Cu at (5.09, 161.5)
- added C52: 1uF, Capacitor_SMD:C_0805_2012Metric, F.Cu at (0.23, 168.7)
- added C53: 100nF, cubesat_rp2040:C_0402_1005Metric, F.Cu at (5.09, 163.5)
- added C54: 10uF, Capacitor_SMD:C_1206_3216Metric, F.Cu at (0.83, 165.5)
- added C55: 100nF, cubesat_rp2040:C_0402_1005Metric, F.Cu at (8.73, 188.2)
- added C56: 1uF, Capacitor_SMD:C_0805_2012Metric, F.Cu at (42.6, 181.3)
- added C57: 1uF, Capacitor_SMD:C_0805_2012Metric, F.Cu at (42.6, 184.3)
- added C58: 100nF, cubesat_rp2040:C_0402_1005Metric, F.Cu at (30.3, 182.7)
- added C59: 100nF, cubesat_rp2040:C_0402_1005Metric, F.Cu at (30.3, 184.7)
- added C60: 100nF, cubesat_rp2040:C_0402_1005Metric, F.Cu at (30.3, 186.7)
- added C61: 100nF, cubesat_rp2040:C_0402_1005Metric, F.Cu at (30.3, 188.7)
- added C62: 100nF, cubesat_rp2040:C_0402_1005Metric, F.Cu at (30.3, 190.6)
- added C63: 100nF, cubesat_rp2040:C_0402_1005Metric, F.Cu at (30.3, 192.6)
- added C64: 100nF, cubesat_rp2040:C_0402_1005Metric, F.Cu at (33.2, 180.8)
- added C65: 100nF, cubesat_rp2040:C_0402_1005Metric, F.Cu at (33.2, 182.7)
- added C66: 100nF, cubesat_rp2040:C_0402_1005Metric, F.Cu at (33.2, 184.7)
- added C67: 100nF, cubesat_rp2040:C_0402_1005Metric, F.Cu at (33.2, 186.7)
- added C68: 100nF, cubesat_rp2040:C_0402_1005Metric, F.Cu at (33.2, 188.7)
- added C69: 100nF, cubesat_rp2040:C_0402_1005Metric, F.Cu at (33.2, 190.6)
- added C70: 100nF, cubesat_rp2040:C_0402_1005Metric, F.Cu at (87.9, 65.2)
- added C71: 100nF, cubesat_rp2040:C_0402_1005Metric, F.Cu at (94.1, 65.9)
- added C72: 4.7nF, cubesat_rp2040:C_0402_1005Metric, F.Cu at (94.1, 62.9)
- added C73: 4.7nF, cubesat_rp2040:C_0402_1005Metric, F.Cu at (94.1, 68.9)
- added C74: 100nF, cubesat_rp2040:C_0402_1005Metric, F.Cu at (33.2, 192.6)
- added C75: 10uF, Capacitor_SMD:C_1206_3216Metric, F.Cu at (0.83, 150.5)
- added C76: 100nF, cubesat_rp2040:C_0402_1005Metric, F.Cu at (5.09, 149.8)
- added C77: 1uF, Capacitor_SMD:C_0805_2012Metric, F.Cu at (0.23, 157.0)
- added C78: 100nF, cubesat_rp2040:C_0402_1005Metric, F.Cu at (5.09, 151.8)
- added C79: 10uF, Capacitor_SMD:C_1206_3216Metric, F.Cu at (0.83, 153.8)
- added C80: 100nF, cubesat_rp2040:C_0402_1005Metric, F.Cu at (-1.79, 188.2)
- added C81: 1uF, Capacitor_SMD:C_0805_2012Metric, F.Cu at (42.6, 187.3)
- added C82: 1uF, Capacitor_SMD:C_0805_2012Metric, F.Cu at (42.6, 190.3)
- added C83: 100nF, cubesat_rp2040:C_0402_1005Metric, F.Cu at (36.1, 180.8)
- added C84: 100nF, cubesat_rp2040:C_0402_1005Metric, F.Cu at (36.1, 182.7)
- added C85: 100nF, cubesat_rp2040:C_0402_1005Metric, F.Cu at (36.1, 184.7)
- added C86: 100nF, cubesat_rp2040:C_0402_1005Metric, F.Cu at (36.1, 186.7)
- added C87: 100nF, cubesat_rp2040:C_0402_1005Metric, F.Cu at (36.1, 188.7)
- added C88: 100nF, cubesat_rp2040:C_0402_1005Metric, F.Cu at (36.1, 190.6)
- added C89: 100nF, cubesat_rp2040:C_0402_1005Metric, F.Cu at (36.1, 192.6)
- added C90: 100nF, cubesat_rp2040:C_0402_1005Metric, F.Cu at (38.9, 180.8)
- added C91: 100nF, cubesat_rp2040:C_0402_1005Metric, F.Cu at (38.9, 182.7)
- added C92: 100nF, cubesat_rp2040:C_0402_1005Metric, F.Cu at (38.9, 184.7)
- added C93: 100nF, cubesat_rp2040:C_0402_1005Metric, F.Cu at (38.9, 186.7)
- added C94: 100nF, cubesat_rp2040:C_0402_1005Metric, F.Cu at (38.9, 188.7)
- added C95: 100nF, cubesat_rp2040:C_0402_1005Metric, F.Cu at (113.3, 65.2)
- added C96: 100nF, cubesat_rp2040:C_0402_1005Metric, F.Cu at (119.5, 65.9)
- added C97: 4.7nF, cubesat_rp2040:C_0402_1005Metric, F.Cu at (119.5, 62.9)
- added C98: 4.7nF, cubesat_rp2040:C_0402_1005Metric, F.Cu at (119.5, 68.9)
- added D1: D_TVS, Diode_SMD:D_0402_1005Metric, F.Cu at (72.9, 59.0)
- added D10: D_TVS, Diode_SMD:D_0402_1005Metric, F.Cu at (65.3, 60.0)
- added D11: D_TVS, Diode_SMD:D_0402_1005Metric, F.Cu at (81.1, 59.0)
- added D12: D_TVS, Diode_SMD:D_0402_1005Metric, F.Cu at (83.1, 59.0)
- added D16: RED, LED_SMD:LED_0402_1005Metric, F.Cu at (113.0, 80.2)
- added D17: RED, LED_SMD:LED_0402_1005Metric, F.Cu at (115.4, 80.2)
- added D18: RED, LED_SMD:LED_0402_1005Metric, F.Cu at (117.8, 80.2)
- added D2: D_TVS, Diode_SMD:D_0402_1005Metric, F.Cu at (70.9, 59.0)
- added D3: D_TVS, Diode_SMD:D_0402_1005Metric, F.Cu at (62.8, 59.0)
- added D4: D_TVS, Diode_SMD:D_0402_1005Metric, F.Cu at (60.8, 59.0)
- added D5: D_TVS, Diode_SMD:D_0402_1005Metric, B.Cu at (57.7, 59.0)
- added D6: D_TVS, Diode_SMD:D_0402_1005Metric, B.Cu at (55.7, 59.0)
- added D7: D_TVS, Diode_SMD:D_0402_1005Metric, B.Cu at (53.2, 60.0)
- added D8: D_TVS, Diode_SMD:D_0402_1005Metric, B.Cu at (55.1, 60.0)
- added D9: D_TVS, Diode_SMD:D_0402_1005Metric, F.Cu at (63.3, 60.0)
- added H1: MountingHole_Pad, MountingHole:MountingHole_3.2mm_M3_Pad_Via, F.Cu at (46.5, 133.8)
- added H2: MountingHole_Pad, MountingHole:MountingHole_3.2mm_M3_Pad_Via, F.Cu at (126.5, 133.8)
- added H3: MountingHole_Pad, MountingHole:MountingHole_3.2mm_M3_Pad_Via, F.Cu at (124.0, 48.1)
- added H4: MountingHole_Pad, MountingHole:MountingHole_3.2mm_M3_Pad_Via, F.Cu at (50.3, 48.1)
- added J1: Conn_01x02, Connector_PinHeader_2.54mm:PinHeader_1x02_P2.54mm_Horizontal, F.Cu at (67.5, 129.0)
- added J2: ESQ-126-39-G-D, cubesat_rp2040:SAMTEC_ESQ-126-39-G-D_CUBESAT, F.Cu at (55.4, 55.7)
- added J3: ESQ-126-39-G-D, cubesat_rp2040:SAMTEC_ESQ-126-39-G-D_CUBESAT, F.Cu at (55.4, 50.6)
- added J6: FTSH-105-01-L-DV-007-K, cubesat_rp2040:SAMTEC_FTSH-105-01-L-DV-007, F.Cu at (33.4, 167.2)
- added J7: FTSH-105-01-L-DV-007-K, cubesat_rp2040:SAMTEC_FTSH-105-01-L-DV-007, F.Cu at (33.4, 175.6)
- added L2: 15uH, Inductor_SMD:L_1210_3225Metric, F.Cu at (2.49, 193.3)
- added L3: 15uH, Inductor_SMD:L_1210_3225Metric, F.Cu at (13.0, 183.3)
- added L4: 15uH, Inductor_SMD:L_1210_3225Metric, F.Cu at (2.49, 183.3)
- added R28: 100kR, cubesat_rp2040:R_0402_1005Metric, F.Cu at (-1.77, 192.2)
- added R29: 100kR, cubesat_rp2040:R_0402_1005Metric, F.Cu at (-1.77, 194.2)
- added R30: 100kR, cubesat_rp2040:R_0402_1005Metric, F.Cu at (-1.77, 196.1)
- added R31: 60R, cubesat_rp2040:R_0402_1005Metric, F.Cu at (68.7, 63.9)
- added R32: 60R, cubesat_rp2040:R_0402_1005Metric, F.Cu at (68.7, 64.9)
- added R33: 60R, cubesat_rp2040:R_0402_1005Metric, F.Cu at (68.7, 66.9)
- added R34: 60R, cubesat_rp2040:R_0402_1005Metric, F.Cu at (68.7, 67.9)
- added R35: 1kR, cubesat_rp2040:R_0402_1005Metric, F.Cu at (21.0, 182.6)
- added R36: 27R, cubesat_rp2040:R_0402_1005Metric, F.Cu at (23.9, 182.6)
- added R37: 27R, cubesat_rp2040:R_0402_1005Metric, F.Cu at (23.9, 184.6)
- added R38: 100kR, cubesat_rp2040:R_0402_1005Metric, F.Cu at (21.0, 184.6)
- added R39: 100kR, cubesat_rp2040:R_0402_1005Metric, F.Cu at (21.0, 186.6)
- added R40: 100kR, cubesat_rp2040:R_0402_1005Metric, F.Cu at (8.75, 182.2)
- added R41: 100kR, cubesat_rp2040:R_0402_1005Metric, F.Cu at (8.75, 184.2)
- added R42: 100kR, cubesat_rp2040:R_0402_1005Metric, F.Cu at (8.75, 186.2)
- added R43: 60R, cubesat_rp2040:R_0402_1005Metric, F.Cu at (94.1, 63.9)
- added R44: 60R, cubesat_rp2040:R_0402_1005Metric, F.Cu at (94.1, 64.9)
- added R45: 60R, cubesat_rp2040:R_0402_1005Metric, F.Cu at (94.1, 66.9)
- added R46: 60R, cubesat_rp2040:R_0402_1005Metric, F.Cu at (94.1, 67.9)
- added R47: 1kR, cubesat_rp2040:R_0402_1005Metric, F.Cu at (23.9, 186.6)
- added R48: 27R, cubesat_rp2040:R_0402_1005Metric, F.Cu at (26.9, 186.6)
- added R49: 27R, cubesat_rp2040:R_0402_1005Metric, F.Cu at (26.9, 188.6)
- added R50: 100kR, cubesat_rp2040:R_0402_1005Metric, F.Cu at (23.9, 188.6)
- added R51: 100kR, cubesat_rp2040:R_0402_1005Metric, F.Cu at (26.9, 182.6)
- added R52: 100kR, cubesat_rp2040:R_0402_1005Metric, F.Cu at (-1.77, 182.2)
- added R53: 100kR, cubesat_rp2040:R_0402_1005Metric, F.Cu at (-1.77, 184.2)
- added R54: 100kR, cubesat_rp2040:R_0402_1005Metric, F.Cu at (-1.77, 186.2)
- added R55: 60R, cubesat_rp2040:R_0402_1005Metric, F.Cu at (119.5, 63.9)
- added R56: 60R, cubesat_rp2040:R_0402_1005Metric, F.Cu at (119.5, 64.9)
- added R57: 60R, cubesat_rp2040:R_0402_1005Metric, F.Cu at (119.5, 66.9)
- added R58: 60R, cubesat_rp2040:R_0402_1005Metric, F.Cu at (119.5, 67.9)
- added R59: 470R, cubesat_rp2040:R_0402_1005Metric, B.Cu at (113.0, 79.2)
- added R60: 470R, cubesat_rp2040:R_0402_1005Metric, B.Cu at (115.4, 79.2)
- added R61: 470R, cubesat_rp2040:R_0402_1005Metric, B.Cu at (117.8, 79.2)
- added R62: 100R, cubesat_rp2040:R_0402_1005Metric, F.Cu at (-16.9, 157.4)
- added R63: 100R, cubesat_rp2040:R_0402_1005Metric, F.Cu at (-6.83, 157.4)
- added R64: 100R, cubesat_rp2040:R_0402_1005Metric, F.Cu at (-27.0, 157.4)
- added R65: 100R, cubesat_rp2040:R_0402_1005Metric, F.Cu at (-16.9, 159.4)
- added R66: 100R, cubesat_rp2040:R_0402_1005Metric, F.Cu at (-6.83, 159.4)
- added R67: 100R, cubesat_rp2040:R_0402_1005Metric, F.Cu at (-27.0, 159.4)
- added U10: RP2040, Package_DFN_QFN:QFN-56-1EP_7x7mm_P0.4mm_EP3.2x3.2mm, F.Cu at (24.2, 167.6)
- added U11: 74LVC1G11, Package_TO_SOT_SMD:SOT-563, F.Cu at (12.1, 187.2)
- added U12: TCAN1048AV-Q1, cubesat_rp2040:SOT1086-2_HVSON14_4.5x3x0.85mm_P0.65mm, F.Cu at (91.0, 65.9)
- added U14: IS25LP128F, Package_SO:SOIC-8_5.275x5.275mm_P1.27mm, F.Cu at (43.7, 174.5)
- added U15: RP2040, Package_DFN_QFN:QFN-56-1EP_7x7mm_P0.4mm_EP3.2x3.2mm, F.Cu at (24.2, 176.9)
- added U16: 74LVC1G11, Package_TO_SOT_SMD:SOT-563, F.Cu at (1.56, 187.2)
- added U17: TCAN1048AV-Q1, cubesat_rp2040:SOT1086-2_HVSON14_4.5x3x0.85mm_P0.65mm, F.Cu at (116.4, 65.9)
- added U18: 74LVC2G38, Package_SO:TSSOP-8_3x3mm_P0.65mm, F.Cu at (115.4, 86.3)
- added U19: 74LVC2G38, Package_SO:TSSOP-8_3x3mm_P0.65mm, F.Cu at (115.4, 91.5)
- added U20: 74LVC2G38, Package_SO:TSSOP-8_3x3mm_P0.65mm, F.Cu at (115.4, 96.7)
- added U21: SN65LVDS1DBV, Package_TO_SOT_SMD:SOT-23-5, F.Cu at (-20.9, 158.8)
- added U22: SN65LVDS1DBV, Package_TO_SOT_SMD:SOT-23-5, F.Cu at (-10.9, 158.8)
- added U23: SN65LVDS1DBV, Package_TO_SOT_SMD:SOT-23-5, F.Cu at (-31.0, 158.8)
- added U24: SN65LVDS2DBV, Package_TO_SOT_SMD:SOT-23-5, F.Cu at (-20.1, 166.9)
- added U25: SN65LVDS2DBV, Package_TO_SOT_SMD:SOT-23-5, F.Cu at (-12.9, 166.9)
- added U26: SN65LVDS2DBV, Package_TO_SOT_SMD:SOT-23-5, F.Cu at (-27.2, 166.9)
- added U27: SN65LVDS2DBV, Package_TO_SOT_SMD:SOT-23-5, F.Cu at (-20.1, 171.5)
- added U28: SN65LVDS2DBV, Package_TO_SOT_SMD:SOT-23-5, F.Cu at (-12.9, 171.5)
- added U29: SN65LVDS2DBV, Package_TO_SOT_SMD:SOT-23-5, F.Cu at (-27.2, 171.5)
- added U6: 74LVC1G11, Package_TO_SOT_SMD:SOT-563, F.Cu at (1.56, 197.1)
- added U7: TCAN1048AV-Q1, cubesat_rp2040:SOT1086-2_HVSON14_4.5x3x0.85mm_P0.65mm, F.Cu at (65.6, 65.9)
- added U9: IS25LP128F, Package_SO:SOIC-8_5.275x5.275mm_P1.27mm, F.Cu at (43.7, 166.8)
- added X1: YSO140TC, cubesat_rp2040:Oscillator_SMD_YXC_YSO140TC_4Pin_3.2x2.5mm, F.Cu at (115.9, 108.7)
- added kibuzzard-66C5B8AD: G***, kibuzzard-66C5B8AD, F.Cu at (85.7, 143.7)
- added kibuzzard-66C5B8B7: G***, kibuzzard-66C5B8B7, F.Cu at (60.2, 143.7)
- added kibuzzard-66C5B8C3: G***, kibuzzard-66C5B8C3, F.Cu at (111.0, 143.7)
- added kibuzzard-66C5B8CC: G***, kibuzzard-66C5B8CC, F.Cu at (57.7, 104.3)
- added kibuzzard-66C5B8D6: G***, kibuzzard-66C5B8D6, F.Cu at (87.2, 130.1)
- added kibuzzard-66C5B8E4: G***, kibuzzard-66C5B8E4, F.Cu at (56.2, 125.7)
- added kibuzzard-66C5B8FA: G***, kibuzzard-66C5B8FA, F.Cu at (78.5, 122.1)
- added kibuzzard-66C5B90B: G***, kibuzzard-66C5B90B, F.Cu at (50.3, 60.3)
- added kibuzzard-66C73F98: G***, kibuzzard-66C73F98, F.Cu at (113.0, 77.4)
- added kibuzzard-66C73FB7: G***, kibuzzard-66C73FB7, F.Cu at (115.4, 77.4)
- added kibuzzard-66C73FBF: G***, kibuzzard-66C73FBF, F.Cu at (117.8, 77.4)
- added kibuzzard-66C73FEB: G***, kibuzzard-66C73FEB, F.Cu at (115.4, 75.8)
- C1: renamed from C101; value 100n -> 100nF; moved to B.Cu
- C10: renamed from C306; value 100n -> 100nF
- C11: renamed from C307; value 100n -> 100nF
- C12: renamed from C308; value 100n -> 100nF
- C13: renamed from C309; value 100n -> 100nF
- C14: renamed from C310; value 100n -> 100nF
- C15: renamed from C311; value 100n -> 100nF
- C16: renamed from C312; value 100n -> 100nF
- C17: renamed from C313; value 100n -> 100nF
- C18: renamed from C314; value 100n -> 100nF
- C19: renamed from C315; value 100n -> 100nF
- C2: renamed from C201; value 1u -> 1uF; moved to B.Cu
- C20: renamed from C316; value 100n -> 100nF
- C21: renamed from C401; value 100n -> 100nF; moved to B.Cu
- C22: renamed from C402; value 10n -> 100nF; moved to B.Cu
- C24: renamed from C501; value 100n -> 100nF
- C3: renamed from C202; value 470n -> 470nF; footprint cubesat_rp2040:C_0402_1005Metric -> Capacitor_SMD:C_0805_2012Metric; moved to B.Cu
- C31: renamed from C502; value 1u -> 1uF; footprint cubesat_rp2040:C_0402_1005Metric -> Capacitor_SMD:C_0805_2012Metric
- C32: renamed from C503; value 1u -> 1uF; footprint cubesat_rp2040:C_0402_1005Metric -> Capacitor_SMD:C_0805_2012Metric
- C33: renamed from C504; value 100n -> 100nF
- C34: renamed from C505; value 100n -> 100nF
- C35: renamed from C506; value 100n -> 100nF
- C36: renamed from C507; value 100n -> 100nF
- C37: renamed from C508; value 100n -> 100nF
- C38: renamed from C509; value 100n -> 100nF
- C39: renamed from C510; value 100n -> 100nF
- C4: renamed from C203; value 470n -> 470nF; footprint cubesat_rp2040:C_0402_1005Metric -> Capacitor_SMD:C_0805_2012Metric; moved to B.Cu
- C40: renamed from C511; value 100n -> 100nF
- C41: renamed from C512; value 100n -> 100nF
- C42: renamed from C513; value 100n -> 100nF
- C43: renamed from C514; value 100n -> 100nF
- C44: renamed from C515; value 100n -> 100nF
- C5: renamed from C204; value 100n -> 100nF; moved to B.Cu
- C6: renamed from C205; value 1u -> 1uF; moved to B.Cu
- C7: renamed from C206; value 10u -> 10uF; footprint Capacitor_SMD:C_0805_2012Metric -> Capacitor_SMD:C_1206_3216Metric
- C8: renamed from C304; value 1u -> 1uF; footprint cubesat_rp2040:C_0402_1005Metric -> Capacitor_SMD:C_0805_2012Metric
- C9: renamed from C305; value 1u -> 1uF; footprint cubesat_rp2040:C_0402_1005Metric -> Capacitor_SMD:C_0805_2012Metric
- J5: renamed from J501; value FTSH-105-01-L-DV-007 -> FTSH-105-01-L-DV-007-K
- L1: renamed from L201; value 10u -> 10uH
- R1: renamed from R101; value 100k -> 100kR; moved to B.Cu
- R10: renamed from R208; moved to B.Cu
- R11: renamed from R301; value 5.1k 10% -> 5.1kR 10%
- R12: renamed from R303; value 5.1k 10% -> 5.1kR 10%
- R13: renamed from R304; value 90.9k 1% -> 90.9kR 1%
- R14: renamed from R305; value 10k 1% -> 10kR 1%
- R15: renamed from R306; value 9.53k 1% -> 9.53kR 1%
- R16: renamed from R307; value 4.7k -> 4.7kR
- R17: renamed from R308; value 4.7k -> 4.7kR
- R18: renamed from R309; value 4.7k -> 4.7kR
- R19: renamed from R310; value 4.7k -> 4.7kR
- R2: renamed from R102; value 10k -> 10kR; moved to B.Cu
- R20: renamed from R311; value 4.7k -> 4.7kR
- R21: renamed from R401; moved to B.Cu
- R22: renamed from R402; value 10k -> 88.7R; moved to B.Cu
- R23: renamed from R510; value 1k -> 1kR; moved to B.Cu
- R26: renamed from R505; value 100k -> 100kR
- R27: renamed from R506; value 100k -> 100kR
- R3: renamed from R201; value 56k -> 56kR; moved to B.Cu
- R4: renamed from R202; value 47k -> 47kR; moved to B.Cu
- R5: renamed from R203; value 100k -> 100kR; moved to B.Cu
- R6: renamed from R204; value 56k -> 56kR; moved to B.Cu
- R7: renamed from R205; value 100k -> 100kR
- R8: renamed from R206; value 47k -> 47kR; moved to B.Cu
- R9: renamed from R207; value 16k -> 16kR; moved to B.Cu
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- renumbered D201 to D13, D302 to D14, D303 to D15, J301 to J4, R508 to R24, R509 to R25, U201 to U1, U502 to U5
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Connections:
- net /RP2040/D+ renamed /RP2040 - Unit A/RP_USB.D+
- net /RP2040/D- renamed /RP2040 - Unit A/RP_USB.D-
- net /RP2040/GPIO0 renamed /RP2040 - Unit A/GPIO0
- net /RP2040/GPIO1 renamed /RP2040 - Unit A/GPIO1
- net /RP2040/GPIO10 renamed /RP2040 - Unit A/CAN_B.STB
- net /RP2040/GPIO15 renamed /RP2040 - Unit A/CAN_A.STB
- net /RP2040/GPIO16 renamed /RP2040 - Unit A/GPIO16
- net /RP2040/GPIO17 renamed /RP2040 - Unit A/GPIO17
- net /RP2040/GPIO18 renamed /RP2040 - Unit A/GPIO18
- net /RP2040/GPIO19 renamed /RP2040 - Unit A/GPIO19
- net /RP2040/GPIO2 renamed /RP2040 - Unit A/GPIO2
- net /RP2040/GPIO20 renamed /RP2040 - Unit A/GPIO20
- net /RP2040/GPIO21 renamed /RP2040 - Unit A/GPIO21
- net /RP2040/GPIO22 renamed /RP2040 - Unit A/GPIO22
- net /RP2040/GPIO23 renamed /RP2040 - Unit A/GPIO23
- net /RP2040/GPIO24 renamed /RP2040 - Unit A/GPIO24
- net /RP2040/GPIO25 renamed /RP2040 - Unit A/GPIO25
- net /RP2040/GPIO29/ADC3 renamed /RP2040 - Unit A/USB_VBUS_DET
- net /RP2040/GPIO3 renamed /RP2040 - Unit A/GPIO3
- net /RP2040/GPIO4 renamed /RP2040 - Unit A/GPIO4
- net /RP2040/GPIO5 renamed /RP2040 - Unit A/GPIO5
- net /RP2040/GPIO6 renamed /RP2040 - Unit A/GPIO6
- net /RP2040/GPIO7 renamed /RP2040 - Unit A/GPIO7
- net /RP2040/GPIO8 renamed /RP2040 - Unit A/GPIO8
- net /RP2040/GPIO9 renamed /RP2040 - Unit A/GPIO9
- net /RP2040/QSPI.SCLK renamed /RP2040 - Unit A/QSPI.SCLK
- net /RP2040/QSPI.SD0 renamed /RP2040 - Unit A/QSPI.SD0
- net /RP2040/QSPI.SD1 renamed /RP2040 - Unit A/QSPI.SD1
- net /RP2040/QSPI.SD2 renamed /RP2040 - Unit A/QSPI.SD2
- net /RP2040/QSPI.SD3 renamed /RP2040 - Unit A/QSPI.SD3
- net /RP2040/QSPI.~{SS} renamed /RP2040 - Unit A/QSPI.~{SS}
- net /RP2040/SWCLK renamed /RP2040 - Unit A/SWCLK
- net /RP2040/SWDIO renamed /RP2040 - Unit A/SWDIO
- C22 pad 2: /Oscillator/F_{out} -> Net-(C22-Pad2)
- C24 pad 1: +3V3 -> /RP2040 - Unit A/+3V3_UNIT
- C31 pad 1: +1V1 -> /RP2040 - Unit A/+1V1_UNIT
- C32 pad 1: +3V3 -> /RP2040 - Unit A/+3V3_UNIT
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Routing:
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- added copper zone on In3.Cu, net +1V1
- added copper zone on In1.Cu, net /+5V
- added copper zone on In2.Cu, net /+5V
- added copper zone on In2.Cu, net /CHARGE
- added copper zone on In2.Cu, net /VBAT
- added copper zone on In2.Cu, net GND
- added copper zone on In3.Cu, net GND
- added copper zone on In4.Cu, net GND
- added copper zone on B.Cu, net VBUS
Other:
- outline, holes or cut-outs redrawn
- copper layers 4 -> 6
- board text added: "0.03048 mm"
- board text added: "0.1088 mm"
- board text added: "0.55 mm"
- board text added: "1.5994 mm"
- board text added: "2116"
- board text added: "3.8"
- board text added: "3313"
- board text added: "4.16"
- board text added: "6"
- board text added: "Black"
- board text added: "Dielectric 4"
- board text added: "Dielectric 5"
- board text added: "In3.Cu"
- board text added: "In4.Cu"
- board text added: "ONLY EDIT THIS RP2040 BLOCK REPLICATE LAYOUT TO THE OTHERS"
- board text removed: "0.01 mm"
- board text removed: "0.017"
- board text removed: "1.265 mm"
- board text removed: "1.5842 mm"
- board text removed: "3.3"
- board text removed: "4"
- board text removed: "Green"
- board text removed: "Rev. ${REVISION}"

Commit message: More work on interfaces
Parts:
- removed D18: RED, LED_SMD:LED_0402_1005Metric
- removed L4: 15uH, Inductor_SMD:L_1210_3225Metric
- removed R57, R58: 60R, cubesat_rp2040:R_0402_1005Metric
- removed R59, R60, R61: 470R, cubesat_rp2040:R_0402_1005Metric
- removed R62, R63, R64, R65, R66, R67: 100R, cubesat_rp2040:R_0402_1005Metric
- removed U24, U25, U26, U27, U28, U29: SN65LVDS2DBV, Package_TO_SOT_SMD:SOT-23-5
- removed kibuzzard-66C5B8AD: G***, kibuzzard-66C5B8AD
- removed kibuzzard-66C5B8B7: G***, kibuzzard-66C5B8B7
- removed kibuzzard-66C5B8C3: G***, kibuzzard-66C5B8C3
- removed kibuzzard-66C5B8CC: G***, kibuzzard-66C5B8CC
- removed kibuzzard-66C5B8D6: G***, kibuzzard-66C5B8D6
- removed kibuzzard-66C5B8E4: G***, kibuzzard-66C5B8E4
- removed kibuzzard-66C5B8FA: G***, kibuzzard-66C5B8FA
- removed kibuzzard-66C5B90B: G***, kibuzzard-66C5B90B
- removed kibuzzard-66C73F98: G***, kibuzzard-66C73F98
- removed kibuzzard-66C73FB7: G***, kibuzzard-66C73FB7
- removed kibuzzard-66C73FBF: G***, kibuzzard-66C73FBF
- removed kibuzzard-66C73FEB: G***, kibuzzard-66C73FEB
- added C100: 1nF, cubesat_rp2040:C_0402_1005Metric, F.Cu at (-53.7, 47.7)
- added C101: 1nF, cubesat_rp2040:C_0402_1005Metric, F.Cu at (-53.7, 49.7)
- added C102: 1nF, cubesat_rp2040:C_0402_1005Metric, F.Cu at (-53.7, 51.7)
- added C103: 1nF, cubesat_rp2040:C_0402_1005Metric, F.Cu at (-53.7, 53.6)
- added C99: 100nF, cubesat_rp2040:C_0402_1005Metric, F.Cu at (-53.7, 45.8)
- added U13: 74LVC1G11, Package_TO_SOT_SMD:SOT-563, F.Cu at (-62.4, 14.4)
- added U3: IS25LP128F, Package_SO:SOIC-8_5.275x5.275mm_P1.27mm, F.Cu at (102.6, 115.6)
- added U8: RP2040, Package_DFN_QFN:QFN-56-1EP_7x7mm_P0.4mm_EP3.2x3.2mm, F.Cu at (-79.0, 39.5)
- C1, C10, C11, C12, C13, C14, C15, C16, C18, C2, C20, C22, C24, C39, C41, C43, C5, D5, D6, D7, D8, R1, R2, R27: moved to F.Cu
- C17: value 100nF -> 15pF; moved to F.Cu
- C19, C40, C44: value 100nF -> 10uF; footprint cubesat_rp2040:C_0402_1005Metric -> Capacitor_SMD:C_1206_3216Metric; moved to F.Cu
- C21, C42: value 100nF -> 1uF; footprint cubesat_rp2040:C_0402_1005Metric -> Capacitor_SMD:C_0805_2012Metric; moved to F.Cu
- C23: value 15pF -> 10uF; footprint cubesat_rp2040:C_0402_1005Metric -> Capacitor_SMD:C_1206_3216Metric; moved to F.Cu
- C25, C29, C50: value 10uF -> 1uF; footprint Capacitor_SMD:C_1206_3216Metric -> Capacitor_SMD:C_0805_2012Metric
- C26, C28, C30: moved to B.Cu
- C27: value 1uF -> 100nF; footprint Capacitor_SMD:C_0805_2012Metric -> cubesat_rp2040:C_0402_1005Metric; moved to B.Cu
- C3: value 470nF -> 1uF; moved to F.Cu
- C31, C32, C52, C56, C57, C77, C81, C82: value 1uF -> 100nF; footprint Capacitor_SMD:C_0805_2012Metric -> cubesat_rp2040:C_0402_1005Metric
- C4: value 470nF -> 100nF; footprint Capacitor_SMD:C_0805_2012Metric -> cubesat_rp2040:C_0402_1005Metric; moved to F.Cu
- C46, C63, C67, C71: value 100nF -> 1uF; footprint cubesat_rp2040:C_0402_1005Metric -> Capacitor_SMD:C_0805_2012Metric
- C47, C48, C72, C73, C97, C98: value 4.7nF -> 100nF
- C54, C75, C79: value 10uF -> 100nF; footprint Capacitor_SMD:C_1206_3216Metric -> cubesat_rp2040:C_0402_1005Metric
- C6, C8, C9: value 1uF -> 100nF; footprint Capacitor_SMD:C_0805_2012Metric -> cubesat_rp2040:C_0402_1005Metric; moved to F.Cu
- C61, C65: value 100nF -> 10uF; footprint cubesat_rp2040:C_0402_1005Metric -> Capacitor_SMD:C_1206_3216Metric
- C7: value 10uF -> 100nF; footprint Capacitor_SMD:C_1206_3216Metric -> cubesat_rp2040:C_0402_1005Metric; moved to F.Cu
- C83, C84, C87, C88, C91, C92: value 100nF -> 4.7nF
- D13: value GREEN -> D_TVS; footprint LED_SMD:LED_0402_1005Metric -> Diode_SMD:D_0402_1005Metric
- D15: value D_TVS -> RED; footprint Diode_SMD:D_0402_1005Metric -> LED_SMD:LED_0402_1005Metric
- L1: value 10uH -> 15uH
- R10: value 470R -> 4.7kR; moved to F.Cu
- R11, R12: value 5.1kR 10% -> 4.7kR
- R13: value 90.9kR 1% -> 4.7kR; moved to F.Cu
- R14: value 10kR 1% -> 33R; moved to F.Cu
- R15: value 9.53kR 1% -> 88.7R; moved to F.Cu
- R16: value 4.7kR -> 1kR; moved to F.Cu
- R17, R18: value 4.7kR -> 27R; moved to F.Cu
- R19, R20: value 4.7kR -> 100kR; moved to F.Cu
- R21: value 33R -> 100kR; moved to F.Cu
- R22: value 88.7R -> 100kR; moved to F.Cu
- R23: value 1kR -> 100kR; moved to F.Cu
- R24: value 27R -> 1kR
- R26: value 100kR -> 27R; moved to F.Cu
- R3: value 56kR -> 5.1kR 10%; moved to F.Cu
- R31: value 60R -> 100kR
- R32: value 60R -> 1kR
- R33, R34: value 60R -> 27R
- R35: value 1kR -> 100kR
- R36, R37: value 27R -> 100kR
- R4: value 47kR -> 5.1kR 10%; moved to F.Cu
- R40, R41, R42, R50, R51: value 100kR -> 60R
- R47: value 1kR -> 60R
- R48, R49: value 27R -> 60R
- R5: value 100kR -> 90.9kR 1%; moved to F.Cu
- R52, R53, R54: value 100kR -> 470R
- R55, R56: value 60R -> 100R
- R6: value 56kR -> 4.7kR; moved to F.Cu
- R7: value 100kR -> 10kR 1%
- R8: value 47kR -> 9.53kR 1%; moved to F.Cu
- R9: value 16kR -> 4.7kR; moved to F.Cu
- U1: value L7983 -> TUSB4041I; footprint cubesat_rp2040:DFN-10-1EP_3x3mm_P0.5mm_EP0.62x0.98mm_Offset0.15mm -> cubesat_rp2040:HTQFP-64-1EP_10x10mm_P0.5mm_EP8x8mm_Mask4.4x4.4mm_ThermalVias
- U10: value RP2040 -> LMR36503MSC3RPERQ1; footprint Package_DFN_QFN:QFN-56-1EP_7x7mm_P0.4mm_EP3.2x3.2mm -> cubesat_rp2040:TI_VQFN-HR_2.1x2.1mm_P0.5mm
- U11: value 74LVC1G11 -> IS25LP128F; footprint Package_TO_SOT_SMD:SOT-563 -> Package_SO:SOIC-8_5.275x5.275mm_P1.27mm
- U12: value TCAN1048AV-Q1 -> RP2040; footprint cubesat_rp2040:SOT1086-2_HVSON14_4.5x3x0.85mm_P0.65mm -> Package_DFN_QFN:QFN-56-1EP_7x7mm_P0.4mm_EP3.2x3.2mm
- U14: value IS25LP128F -> TCAN1048AV-Q1; footprint Package_SO:SOIC-8_5.275x5.275mm_P1.27mm -> cubesat_rp2040:SOT1086-2_HVSON14_4.5x3x0.85mm_P0.65mm
- U15: value RP2040 -> TCAN1048AV-Q1; footprint Package_DFN_QFN:QFN-56-1EP_7x7mm_P0.4mm_EP3.2x3.2mm -> cubesat_rp2040:SOT1086-2_HVSON14_4.5x3x0.85mm_P0.65mm
- U16: value 74LVC1G11 -> TCAN1048AV-Q1; footprint Package_TO_SOT_SMD:SOT-563 -> cubesat_rp2040:SOT1086-2_HVSON14_4.5x3x0.85mm_P0.65mm
- U17: value TCAN1048AV-Q1 -> 74LVC2G38; footprint cubesat_rp2040:SOT1086-2_HVSON14_4.5x3x0.85mm_P0.65mm -> Package_SO:TSSOP-8_3x3mm_P0.65mm
- U2: value TUSB4041I -> LMR36503MSC3RPERQ1; footprint cubesat_rp2040:HTQFP-64-1EP_10x10mm_P0.5mm_EP8x8mm_Mask4.4x4.4mm_ThermalVias -> cubesat_rp2040:TI_VQFN-HR_2.1x2.1mm_P0.5mm
- U20: value 74LVC2G38 -> SN65LVDS1DBV; footprint Package_SO:TSSOP-8_3x3mm_P0.65mm -> Package_TO_SOT_SMD:SOT-23-5
- U22, U23: value SN65LVDS1DBV -> SN65LVDS2DBV
- U4: value IS25LP128F -> RP2040; footprint Package_SO:SOIC-8_5.275x5.275mm_P1.27mm -> Package_DFN_QFN:QFN-56-1EP_7x7mm_P0.4mm_EP3.2x3.2mm
- U5: value RP2040 -> 74LVC1G11; footprint Package_DFN_QFN:QFN-56-1EP_7x7mm_P0.4mm_EP3.2x3.2mm -> Package_TO_SOT_SMD:SOT-563
- U6: value 74LVC1G11 -> LMR36503MSC3RPERQ1; footprint Package_TO_SOT_SMD:SOT-563 -> cubesat_rp2040:TI_VQFN-HR_2.1x2.1mm_P0.5mm
- U7: value TCAN1048AV-Q1 -> IS25LP128F; footprint cubesat_rp2040:SOT1086-2_HVSON14_4.5x3x0.85mm_P0.65mm -> Package_SO:SOIC-8_5.275x5.275mm_P1.27mm
- U9: value IS25LP128F -> 74LVC1G11; footprint Package_SO:SOIC-8_5.275x5.275mm_P1.27mm -> Package_TO_SOT_SMD:SOT-563
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Connections:
- net /+5V renamed /Cubesat System Bus/+5V
- net /CHARGE renamed /Cubesat System Bus/CHARGE
- net /RP2040 - Unit A/LVDS_A_TX.N renamed /LVDS/LVDS_TX_B.N
- net /RP2040 - Unit A/LVDS_A_TX.P renamed /LVDS/LVDS_TX_B.P
- net /UART_D.D+ renamed /Cubesat System Bus/UART_D.D+
- net /UART_D.D- renamed /Cubesat System Bus/UART_D.D-
- net /VBAT renamed /Cubesat System Bus/VBAT
- C1 pad 1: /~{RESET} -> /~{USR_RESET}
- C11 pad 1: +1V1 -> +3V3
- C12 pad 1: +1V1 -> +3V3
- C13 pad 1: +1V1 -> +3V3
- C14 pad 1: +1V1 -> +3V3
- C15 pad 1: +1V1 -> Net-(X1-Vdd)
- C16 pad 1: +1V1 -> Net-(X1-OUT)
- C16 pad 2: GND -> Net-(C16-Pad2)
- C17 pad 1: +3V3 -> GND
- C17 pad 2: GND -> /Oscillator/24M0_CLK
- C18 pad 1: +3V3 -> /RP2040 - Unit A/+3V3_UNIT
- C19 pad 1: +3V3 -> VBUS
- C2 pad 1: VBUS -> +1V1
- C20 pad 1: +3V3 -> VBUS
- C21 pad 1: Net-(X1-Vdd) -> Net-(U2-RT)
- C22 pad 1: Net-(X1-OUT) -> /RP2040 - Unit A/BOOT
- C22 pad 2: Net-(C22-Pad2) -> /RP2040 - Unit A/SW
- C23 pad 1: GND -> /RP2040 - Unit A/+3V3_UNIT
- C23 pad 2: /Oscillator/24M0_CLK -> GND
- C25 pad 1: /RP2040 - Unit A/VIN -> /RP2040 - Unit A/+1V1_UNIT
- C26 pad 1: /RP2040 - Unit A/VIN -> /RP2040 - Unit A/+1V1_UNIT
- C27 pad 1: Net-(U3-RT) -> /RP2040 - Unit A/+1V1_UNIT
- C28 pad 1: /RP2040 - Unit A/BOOT -> /RP2040 - Unit A/+1V1_UNIT
- C28 pad 2: /RP2040 - Unit A/SW -> GND
- C3 pad 1: /Power/VCC -> +3V3
- C31 pad 1: /RP2040 - Unit A/+1V1_UNIT -> /RP2040 - Unit A/+3V3_UNIT
- C33 pad 1: /RP2040 - Unit A/+1V1_UNIT -> /RP2040 - Unit A/+3V3_UNIT
- C34 pad 1: /RP2040 - Unit A/+1V1_UNIT -> /RP2040 - Unit A/+3V3_UNIT
- C35 pad 1: /RP2040 - Unit A/+1V1_UNIT -> /RP2040 - Unit A/+3V3_UNIT
- C39 pad 1: /RP2040 - Unit A/+3V3_UNIT -> /RP2040 - Unit B/+3V3_UNIT
- C4 pad 1: /Power/EN/UVLO -> +1V1
- C40 pad 1: /RP2040 - Unit A/+3V3_UNIT -> VBUS
- C41 pad 1: /RP2040 - Unit A/+3V3_UNIT -> VBUS
- C42 pad 1: /RP2040 - Unit A/+3V3_UNIT -> Net-(U6-RT)
- C43 pad 1: /RP2040 - Unit A/+3V3_UNIT -> /RP2040 - Unit B/BOOT
- C43 pad 2: GND -> /RP2040 - Unit B/SW
- C44 pad 1: /RP2040 - Unit A/+3V3_UNIT -> /RP2040 - Unit B/+3V3_UNIT
- C45 pad 1: +5V -> /RP2040 - Unit B/+3V3_UNIT
- C46 pad 1: +3V3 -> /RP2040 - Unit B/+1V1_UNIT
- C47 pad 1: GND -> /RP2040 - Unit B/+1V1_UNIT
- C47 pad 2: Net-(C47-Pad2) -> GND
- C48 pad 1: GND -> /RP2040 - Unit B/+1V1_UNIT
- C48 pad 2: Net-(C48-Pad2) -> GND
- C49 pad 1: /RP2040 - Unit B/+3V3_UNIT -> /RP2040 - Unit B/+1V1_UNIT
- C5 pad 1: +3V3 -> +1V1
- C50 pad 1: /RP2040 - Unit B/VIN -> /RP2040 - Unit B/+3V3_UNIT
- C51 pad 1: /RP2040 - Unit B/VIN -> /RP2040 - Unit B/+3V3_UNIT
- C52 pad 1: Net-(U8-RT) -> /RP2040 - Unit B/+3V3_UNIT
- C53 pad 1: /RP2040 - Unit B/BOOT -> /RP2040 - Unit B/+3V3_UNIT
- C53 pad 2: /RP2040 - Unit B/SW -> GND
- C56 pad 1: /RP2040 - Unit B/+1V1_UNIT -> /RP2040 - Unit B/+3V3_UNIT
- C58 pad 1: /RP2040 - Unit B/+1V1_UNIT -> /RP2040 - Unit B/+3V3_UNIT
- C59 pad 1: /RP2040 - Unit B/+1V1_UNIT -> /RP2040 - Unit B/+3V3_UNIT
- C6 pad 1: +3V3 -> +1V1
- C60 pad 1: /RP2040 - Unit B/+1V1_UNIT -> /RP2040 - Unit C/+3V3_UNIT
- C61 pad 1: /RP2040 - Unit B/+3V3_UNIT -> VBUS
- C62 pad 1: /RP2040 - Unit B/+3V3_UNIT -> VBUS
- C63 pad 1: /RP2040 - Unit B/+3V3_UNIT -> Net-(U10-RT)
- C64 pad 1: /RP2040 - Unit B/+3V3_UNIT -> /RP2040 - Unit C/BOOT
- C64 pad 2: GND -> /RP2040 - Unit C/SW
- C65 pad 1: /RP2040 - Unit B/+3V3_UNIT -> /RP2040 - Unit C/+3V3_UNIT
- C66 pad 1: /RP2040 - Unit B/+3V3_UNIT -> /RP2040 - Unit C/+3V3_UNIT
- C67 pad 1: /RP2040 - Unit B/+3V3_UNIT -> /RP2040 - Unit C/+1V1_UNIT
- C68 pad 1: /RP2040 - Unit B/+3V3_UNIT -> /RP2040 - Unit C/+1V1_UNIT
- C69 pad 1: /RP2040 - Unit B/+3V3_UNIT -> /RP2040 - Unit C/+1V1_UNIT
- C7 pad 1: VBUS -> +1V1
- C70 pad 1: +5V -> /RP2040 - Unit C/+1V1_UNIT
- C71 pad 1: +3V3 -> /RP2040 - Unit C/+3V3_UNIT
- C72 pad 1: GND -> /RP2040 - Unit C/+3V3_UNIT
- C72 pad 2: Net-(C72-Pad2) -> GND
- C73 pad 1: GND -> /RP2040 - Unit C/+3V3_UNIT
- C73 pad 2: Net-(C73-Pad2) -> GND
- C75 pad 1: /RP2040 - Unit C/VIN -> /RP2040 - Unit C/+3V3_UNIT
- C76 pad 1: /RP2040 - Unit C/VIN -> /RP2040 - Unit C/+3V3_UNIT
- C77 pad 1: Net-(U13-RT) -> /RP2040 - Unit C/+3V3_UNIT
- C78 pad 1: /RP2040 - Unit C/BOOT -> /RP2040 - Unit C/+3V3_UNIT
- C78 pad 2: /RP2040 - Unit C/SW -> GND
- C81 pad 1: /RP2040 - Unit C/+1V1_UNIT -> +5V
- C82 pad 1: /RP2040 - Unit C/+3V3_UNIT -> +3V3
- C83 pad 1: /RP2040 - Unit C/+1V1_UNIT -> GND
- C83 pad 2: GND -> Net-(C83-Pad2)
- C84 pad 1: /RP2040 - Unit C/+1V1_UNIT -> GND
- C84 pad 2: GND -> Net-(C84-Pad2)
- C85 pad 1: /RP2040 - Unit C/+1V1_UNIT -> +5V
- C86 pad 1: /RP2040 - Unit C/+3V3_UNIT -> +3V3
- C87 pad 1: /RP2040 - Unit C/+3V3_UNIT -> GND
- C87 pad 2: GND -> Net-(C87-Pad2)
- C88 pad 1: /RP2040 - Unit C/+3V3_UNIT -> GND
- C88 pad 2: GND -> Net-(C88-Pad2)
- C89 pad 1: /RP2040 - Unit C/+3V3_UNIT -> +5V
- C9 pad 1: +3V3 -> +1V1
- C90 pad 1: /RP2040 - Unit C/+3V3_UNIT -> +3V3
- C91 pad 1: /RP2040 - Unit C/+3V3_UNIT -> GND
- C91 pad 2: GND -> Net-(C91-Pad2)
- C92 pad 1: /RP2040 - Unit C/+3V3_UNIT -> GND
- C92 pad 2: GND -> Net-(C92-Pad2)
- C93 pad 1: /RP2040 - Unit C/+3V3_UNIT -> +3V3
- C94 pad 1: /RP2040 - Unit C/+3V3_UNIT -> +3V3
- C95 pad 1: +5V -> +3V3
- C96 pad 1: +3V3 -> /LVDS/+3V3_UNIT
- C97 pad 1: GND -> /LVDS/+3V3_UNIT
- C97 pad 2: Net-(C97-Pad2) -> GND
- C98 pad 1: GND -> /LVDS/+3V3_UNIT
- C98 pad 2: Net-(C98-Pad2) -> GND
- D1 pad 2: /UART_C.D- -> /CAN PHY - UNIT A/CAN_A.P
- D10 pad 2: /UART_B.D- -> /Cubesat System Bus/UART_C.D-
- D13 pad 1: Net-(D13-K) -> GND
- D13 pad 2: /Power/~{RESET} -> /USB/USB_UP.D+
- D14 pad 2: /USB/USB_UP.D+ -> /USB/USB_UP.D-
- D15 pad 1: GND -> /TMR/~{TMR_RESET_A}
- D15 pad 2: /USB/USB_UP.D- -> Net-(D15-A)
- D16 pad 1: /TMR voting/TMR_RESET_A -> /TMR/~{TMR_RESET_B}
- D17 pad 1: /TMR voting/TMR_RESET_B -> /TMR/~{TMR_RESET_C}
- D2 pad 2: /UART_C.D+ -> /CAN PHY - UNIT A/CAN_A.N
- D3 pad 2: /UART_A.D- -> /CAN PHY - UNIT A/CAN_B.P
- D4 pad 2: /UART_A.D+ -> /CAN PHY - UNIT A/CAN_B.N
- D5 pad 2: /CAN_A.P -> /Cubesat System Bus/UART_A.D+
- D6 pad 2: /CAN_A.N -> /Cubesat System Bus/UART_A.D-
- D7 pad 2: /CAN_B.N -> /Cubesat System Bus/UART_B.D+
- D8 pad 2: /CAN_B.P -> /Cubesat System Bus/UART_B.D-
- D9 pad 2: /UART_B.D+ -> /Cubesat System Bus/UART_C.D+
- J1 pad 1: /~{USB_BOOT} -> /BOOTSEL
- J2 pad 01: /CAN_A.N -> /CAN PHY - UNIT A/CAN_A.N
- J2 pad 02: /CAN_B.N -> /CAN PHY - UNIT A/CAN_B.N
- J2 pad 03: /CAN_A.P -> /CAN PHY - UNIT A/CAN_A.P
- J2 pad 04: /CAN_B.P -> /CAN PHY - UNIT A/CAN_B.P
- J2 pad 05: /UART_A.D+ -> /Cubesat System Bus/UART_A.D+
- J2 pad 06: /UART_B.D+ -> /Cubesat System Bus/UART_B.D+
- J2 pad 07: /UART_A.D- -> /Cubesat System Bus/UART_A.D-
- J2 pad 08: /UART_B.D- -> /Cubesat System Bus/UART_B.D-
- J2 pad 13: /UART_C.D+ -> /Cubesat System Bus/UART_C.D+
- J2 pad 15: /UART_C.D- -> /Cubesat System Bus/UART_C.D-
- J2 pad 27: +3V3 -> /Cubesat System Bus/+3V3
- J2 pad 28: +3V3 -> /Cubesat System Bus/+3V3
- J5 pad 10: /RP2040 - Unit A/~{USR_RESET} -> /~{USR_RESET}
- J6 pad 10: /RP2040 - Unit B/~{USR_RESET} -> /~{USR_RESET}
- J7 pad 10: /RP2040 - Unit C/~{USR_RESET} -> /~{USR_RESET}
- L1 pad 1: /Power/LX -> /RP2040 - Unit A/SW
- L1 pad 2: +3V3 -> /RP2040 - Unit A/+3V3_UNIT
- L2 pad 1: /RP2040 - Unit A/SW -> /RP2040 - Unit B/SW
- L2 pad 2: /RP2040 - Unit A/+3V3_UNIT -> /RP2040 - Unit B/+3V3_UNIT
- L3 pad 1: /RP2040 - Unit B/SW -> /RP2040 - Unit C/SW
- L3 pad 2: /RP2040 - Unit B/+3V3_UNIT -> /RP2040 - Unit C/+3V3_UNIT
- R10 pad 1: GND -> /USB/PWRCTL4/BATEN4
- R10 pad 2: Net-(D13-K) -> GND
- R11 pad 1: /USB/USB_UP.CC2 -> /USB/PWRCTL3/BATEN3
- R12 pad 1: /USB/USB_UP.CC1 -> /USB/PWRCTL2/BATEN2
- R13 pad 1: VBUS -> /USB/PWRCTL1/BATEN1
- R13 pad 2: /USB/USB_VBUS -> GND
- R14 pad 1: /USB/USB_VBUS -> +3V3
- R14 pad 2: GND -> Net-(X1-Vdd)
- R15 pad 1: Net-(U2-USB_R1) -> Net-(C16-Pad2)
- R15 pad 2: GND -> /Oscillator/24M0_CLK
- R16 pad 1: Net-(U2-GANGED/SMBA2/HS_UP) -> /RP2040 - Unit A/QSPI.~{SS}
- R16 pad 2: GND -> /BOOTSEL
- R17 pad 1: /USB/PWRCTL4/BATEN4 -> /RP2040 - Unit A/USB.D+
- R17 pad 2: GND -> /RP2040 - Unit A/RP_USB.D+
- R18 pad 1: /USB/PWRCTL3/BATEN3 -> /RP2040 - Unit A/USB.D-
- R18 pad 2: GND -> /RP2040 - Unit A/RP_USB.D-
- R19 pad 1: /USB/PWRCTL2/BATEN2 -> /RP2040 - Unit A/SWDIO
- R19 pad 2: GND -> /RP2040 - Unit A/+3V3_UNIT
- R2 pad 1: /~{RESET} -> /~{USR_RESET}
- R20 pad 1: /USB/PWRCTL1/BATEN1 -> GND
- R20 pad 2: GND -> /RP2040 - Unit A/SWCLK
- R21 pad 1: +3V3 -> /RP2040 - Unit A/+3V3_UNIT
- R21 pad 2: Net-(X1-Vdd) -> /~{USR_RESET}
- R22 pad 1: Net-(C22-Pad2) -> /RP2040 - Unit A/+3V3_UNIT
- R22 pad 2: /Oscillator/24M0_CLK -> /RP2040 - Unit A/~{PWR_RESET}
- R23 pad 1: /RP2040 - Unit A/QSPI.~{SS} -> /RP2040 - Unit A/+3V3_UNIT
- R23 pad 2: /~{USB_BOOT} -> /TMR/~{TMR_RESET_A}
- R24 pad 1: /RP2040 - Unit A/USB.D+ -> /RP2040 - Unit B/QSPI.~{SS}
- R24 pad 2: /RP2040 - Unit A/RP_USB.D+ -> /BOOTSEL
- R25 pad 1: /RP2040 - Unit A/USB.D- -> /RP2040 - Unit B/USB.D+
- R25 pad 2: /RP2040 - Unit A/RP_USB.D- -> /RP2040 - Unit B/RP_USB.D+
- R26 pad 1: /RP2040 - Unit A/SWDIO -> /RP2040 - Unit B/USB.D-
- R26 pad 2: /RP2040 - Unit A/+3V3_UNIT -> /RP2040 - Unit B/RP_USB.D-
- R27 pad 1: GND -> /RP2040 - Unit B/SWDIO
- R27 pad 2: /RP2040 - Unit A/SWCLK -> /RP2040 - Unit B/+3V3_UNIT
- R28 pad 1: /RP2040 - Unit A/+3V3_UNIT -> GND
- R28 pad 2: /RP2040 - Unit A/~{USR_RESET} -> /RP2040 - Unit B/SWCLK
- R29 pad 1: /RP2040 - Unit A/+3V3_UNIT -> /RP2040 - Unit B/+3V3_UNIT
- R29 pad 2: /RP2040 - Unit A/~{PWR_RESET} -> /~{USR_RESET}
- R3 pad 1: /Power/FSW -> /USB/USB_UP.CC2
- R3 pad 2: /Power/VCC -> GND
- R30 pad 1: /RP2040 - Unit A/+3V3_UNIT -> /RP2040 - Unit B/+3V3_UNIT
- R30 pad 2: /RP2040 - Unit A/~{TMR_RESET} -> /RP2040 - Unit B/~{PWR_RESET}
- R31 pad 1: /CAN_A.P -> /RP2040 - Unit B/+3V3_UNIT
- R31 pad 2: Net-(C47-Pad2) -> /TMR/~{TMR_RESET_B}
- R32 pad 1: /CAN_A.N -> /RP2040 - Unit C/QSPI.~{SS}
- R32 pad 2: Net-(C47-Pad2) -> /BOOTSEL
- R33 pad 1: /CAN_B.P -> /RP2040 - Unit C/USB.D+
- R33 pad 2: Net-(C48-Pad2) -> /RP2040 - Unit C/RP_USB.D+
- R34 pad 1: /CAN_B.N -> /RP2040 - Unit C/USB.D-
- R34 pad 2: Net-(C48-Pad2) -> /RP2040 - Unit C/RP_USB.D-
- R35 pad 1: /RP2040 - Unit B/QSPI.~{SS} -> /RP2040 - Unit C/SWDIO
- R35 pad 2: /~{USB_BOOT} -> /RP2040 - Unit C/+3V3_UNIT
- R36 pad 1: /RP2040 - Unit B/USB.D+ -> GND
- R36 pad 2: /RP2040 - Unit B/RP_USB.D+ -> /RP2040 - Unit C/SWCLK
- R37 pad 1: /RP2040 - Unit B/USB.D- -> /RP2040 - Unit C/+3V3_UNIT
- R37 pad 2: /RP2040 - Unit B/RP_USB.D- -> /~{USR_RESET}
- R38 pad 1: /RP2040 - Unit B/SWDIO -> /RP2040 - Unit C/+3V3_UNIT
- R38 pad 2: /RP2040 - Unit B/+3V3_UNIT -> /RP2040 - Unit C/~{PWR_RESET}
- R39 pad 1: GND -> /RP2040 - Unit C/+3V3_UNIT
- R39 pad 2: /RP2040 - Unit B/SWCLK -> /TMR/~{TMR_RESET_C}
- R4 pad 1: /LNM_ENABLE -> /USB/USB_UP.CC1
- R40 pad 1: /RP2040 - Unit B/+3V3_UNIT -> /CAN PHY - UNIT A/CAN_A.P
- R40 pad 2: /RP2040 - Unit B/~{USR_RESET} -> Net-(C83-Pad2)
- R41 pad 1: /RP2040 - Unit B/+3V3_UNIT -> /CAN PHY - UNIT A/CAN_A.N
- R41 pad 2: /RP2040 - Unit B/~{PWR_RESET} -> Net-(C83-Pad2)
- R42 pad 1: /RP2040 - Unit B/+3V3_UNIT -> /CAN PHY - UNIT A/CAN_B.P
- R42 pad 2: /RP2040 - Unit B/~{TMR_RESET} -> Net-(C84-Pad2)
- R43 pad 1: /CAN_A.P -> /CAN PHY - UNIT A/CAN_B.N
- R43 pad 2: Net-(C72-Pad2) -> Net-(C84-Pad2)
- R44 pad 1: /CAN_A.N -> /CAN PHY - UNIT A/CAN_A.P
- R44 pad 2: Net-(C72-Pad2) -> Net-(C87-Pad2)
- R45 pad 1: /CAN_B.P -> /CAN PHY - UNIT A/CAN_A.N
- R45 pad 2: Net-(C73-Pad2) -> Net-(C87-Pad2)
- R46 pad 1: /CAN_B.N -> /CAN PHY - UNIT A/CAN_B.P
- R46 pad 2: Net-(C73-Pad2) -> Net-(C88-Pad2)
- R47 pad 1: /RP2040 - Unit C/QSPI.~{SS} -> /CAN PHY - UNIT A/CAN_B.N
- R47 pad 2: /~{USB_BOOT} -> Net-(C88-Pad2)
- R48 pad 1: /RP2040 - Unit C/USB.D+ -> /CAN PHY - UNIT A/CAN_A.P
- R48 pad 2: /RP2040 - Unit C/RP_USB.D+ -> Net-(C91-Pad2)
- R49 pad 1: /RP2040 - Unit C/USB.D- -> /CAN PHY - UNIT A/CAN_A.N
- R49 pad 2: /RP2040 - Unit C/RP_USB.D- -> Net-(C91-Pad2)
- R5 pad 1: /Power/EN/UVLO -> VBUS
- R5 pad 2: VBUS -> /USB/USB_VBUS
- R50 pad 1: /RP2040 - Unit C/SWDIO -> /CAN PHY - UNIT A/CAN_B.P
- R50 pad 2: /RP2040 - Unit C/+3V3_UNIT -> Net-(C92-Pad2)
- R51 pad 1: GND -> /CAN PHY - UNIT A/CAN_B.N
- R51 pad 2: /RP2040 - Unit C/SWCLK -> Net-(C92-Pad2)
- R52 pad 1: /RP2040 - Unit C/+3V3_UNIT -> +3V3
- R52 pad 2: /RP2040 - Unit C/~{USR_RESET} -> Net-(D15-A)
- R53 pad 1: /RP2040 - Unit C/+3V3_UNIT -> +3V3
- R53 pad 2: /RP2040 - Unit C/~{PWR_RESET} -> Net-(D16-A)
- R54 pad 1: /RP2040 - Unit C/+3V3_UNIT -> +3V3
- R54 pad 2: /RP2040 - Unit C/~{TMR_RESET} -> Net-(D17-A)
- R55 pad 1: /CAN_A.P -> /LVDS/LVDS_RX_A.P
- R55 pad 2: Net-(C97-Pad2) -> /LVDS/LVDS_RX_A.N
- R56 pad 1: /CAN_A.N -> /LVDS/LVDS_RX_B.P
- R56 pad 2: Net-(C97-Pad2) -> /LVDS/LVDS_RX_B.N
- R6 pad 1: GND -> Net-(U1-GANGED/SMBA2/HS_UP)
- R6 pad 2: /Power/EN/UVLO -> GND
- R7 pad 1: VBUS -> /USB/USB_VBUS
- R7 pad 2: /Power/~{RESET} -> GND
- R8 pad 1: +3V3 -> Net-(U1-USB_R1)
- R8 pad 2: /Power/FB -> GND
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Routing:
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- removed copper zone on In3.Cu, net +1V1
- removed copper zone on In2.Cu, net +3V3
- removed copper zone on In1.Cu, net /Cubesat System Bus/+5V
- removed copper zone on In2.Cu, net /Cubesat System Bus/+5V
- removed copper zone on In2.Cu, net /Cubesat System Bus/CHARGE
- removed copper zone on In2.Cu, net /Cubesat System Bus/VBAT
- removed copper zone on B.Cu, net VBUS
