File: reset.kicad_sch (KiCad schematic)
At the start: 4 parts, among them SW1 SW_Push

Commit message: Update footprints, route switching regulator circuit block
Parts:
- SW1: footprint (none) -> Button_Switch_SMD:SW_Push_1P1T_NO_6x6mm_H9.5mm
Changed lines of the file:
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@@
 			)
 		)
-		(property "Footprint" ""
+		(property "Footprint" "Button_Switch_SMD:SW_Push_1P1T_NO_6x6mm_H9.5mm"
 			(at 129.54 102.87 0)
 			(effects

Commit message: Update README, change footprints
Parts:
- SW1: footprint Button_Switch_SMD:SW_Push_1P1T_NO_6x6mm_H9.5mm -> Button_Switch_SMD:SW_SPST_B3U-1000P
Changed lines of the file:
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@@
 			)
 		)
-		(property "Footprint" "Button_Switch_SMD:SW_Push_1P1T_NO_6x6mm_H9.5mm"
+		(property "Footprint" "Button_Switch_SMD:SW_SPST_B3U-1000P"
 			(at 129.54 102.87 0)
 			(effects

Commit message: Big update, bad commit messsage :)
Parts:
- C901: renamed from C22; value C_Small -> C; footprint Capacitor_SMD:C_0402_1005Metric -> cubesat_rp2040:C_0402_1005Metric; symbol Device:C_Small -> Device:C
- R901: renamed from R15; footprint Resistor_SMD:R_0402_1005Metric -> cubesat_rp2040:R_0402_1005Metric
- R902: renamed from R16; footprint Resistor_SMD:R_0402_1005Metric -> cubesat_rp2040:R_0402_1005Metric
- renumbered SW1 to SW901
Connections:
- net RUN renamed ~{RESET}
Other:
- company: (none) -> Magnus Oksbøl Therkelsen
- title: (none) -> CubeSat RP2040 Board
Changed lines of the file:
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@@
 	(generator_version "8.0")
 	(paper "A4")
+	(title_block
+		(title "CubeSat RP2040 Board")
+		(rev "1")
+		(company "Magnus Oksbøl Therkelsen")
+		(comment 1 "Author: Magnus Oksbøl Therkelsen")
+		(comment 2 "Checked by: ")
+	)
+	(junction
+		(at 152.4 95.25)
+		(diameter 0)
+		(color 0 0 0 0)
+	)
 	(junction
 		(at 157.48 95.25)
@@
 		(color 0 0 0 0)
 	)
-	(junction
-		(at 152.4 95.25)
-		(diameter 0)
-		(color 0 0 0 0)
+	(wire
+		(pts
+			(xy 152.4 95.25) (xy 157.48 95.25)
+		)
+		(stroke
+			(width 0)
+			(type default)
+		)
+	)
+	(wire
+		(pts
+			(xy 134.62 97.79) (xy 134.62 95.25)
+		)
+		(stroke
+			(width 0)
+			(type default)
+		)
+	)
+	(wire
+		(pts
+			(xy 134.62 95.25) (xy 139.7 95.25)
+		)
+		(stroke
+			(width 0)
+			(type default)
+		)
+	)
+	(wire
+		(pts
+			(xy 147.32 95.25) (xy 152.4 95.25)
+		)
+		(stroke
+			(width 0)
+			(type default)
+		)
+	)
+	(wire
+		(pts
+			(xy 152.4 92.71) (xy 152.4 95.25)
+		)
+		(stroke
+			(width 0)
+			(type default)
+		)
+	)
+	(wire
+		(pts
+			(xy 134.62 107.95) (xy 134.62 110.49)
+		)
+		(stroke
+			(width 0)
+			(type default)
+		)
+	)
+	(wire
+		(pts
+			(xy 157.48 106.68) (xy 157.48 110.49)
+		)
+		(stroke
+			(width 0)
+			(type default)
+		)
+	)
+	(wire
+		(pts
+			(xy 157.48 95.25) (xy 157.48 99.06)
+		)
+		(stroke
+			(width 0)
+			(type default)
+		)
 	)
 	(wire
@@
 	(wire
 		(pts
-			(xy 134.62 97.79) (xy 134.62 95.25)
-		)
-		(stroke
-			(width 0)
-			(type default)
-		)
-	)
-	(wire
-		(pts
-			(xy 157.48 95.25) (xy 157.48 100.33)
-		)
-		(stroke
-			(width 0)
-			(type default)
-		)
-	)
-	(wire
-		(pts
-			(xy 134.62 95.25) (xy 139.7 95.25)
-		)
-		(stroke
-			(width 0)
-			(type default)
-		)
-	)
-	(wire
-		(pts
-			(xy 147.32 95.25) (xy 152.4 95.25)
-		)
-		(stroke
-			(width 0)
-			(type default)
-		)
-	)
-	(wire
-		(pts
-			(xy 152.4 92.71) (xy 152.4 95.25)
-		)
-		(stroke
-			(width 0)
-			(type default)
-		)
-	)
-	(wire
-		(pts
-			(xy 134.62 107.95) (xy 134.62 110.49)
-		)
-		(stroke
-			(width 0)
-			(type default)
-		)
-	)
-	(wire
-		(pts
-			(xy 157.48 105.41) (xy 157.48 110.49)
-		)
-		(stroke
-			(width 0)
-			(type default)
-		)
-	)
-	(wire
-		(pts
-			(xy 152.4 95.25) (xy 157.48 95.25)
-		)
-		(stroke
-			(width 0)
-			(type default)
-		)
-	)
-	(wire
-		(pts
 			(xy 152.4 82.55) (xy 152.4 85.09)
 		)
@@
 		)
 	)
-	(hierarchical_label "RUN"
+	(hierarchical_label "~{RESET}"
 		(shape output)
 		(at 165.1 95.25 0)
@@
 	)
 	(symbol
-		(lib_id "Device:C_Small")
+		(lib_id "Device:C")
 		(at 157.48 102.87 0)
 		(unit 1)
@@
 		(dnp no)
 		(fields_autoplaced yes)
-		(property "Reference" "C22"
-			(at 160.02 101.6063 0)
+		(property "Reference" "C901"
+			(at 161.29 101.5999 0)
 			(effects
 				(font
@@
 			)
 		)
-		(property "Value" "C_Small"
-			(at 160.02 104.1463 0)
+		(property "Value" "C"
+			(at 161.29 104.1399 0)
 			(effects
 				(font
@@
 			)
 		)
-		(property "Footprint" "Capacitor_SMD:C_0402_1005Metric"
-			(at 157.48 102.87 0)
+		(property "Footprint" "cubesat_rp2040:C_0402_1005Metric"
+			(at 158.4452 106.68 0)
 			(effects
 				(font
@@
 			)
 		)
-		(property "Description" "Unpolarized capacitor, small symbol"
+		(property "Description" "Unpolarized capacitor"
 			(at 157.48 102.87 0)
 			(effects
@@
 			(project "cubesat_rp2040"
 				(path "/5511013b-c214-40ba-8960-f470f52474f8/1dd649c8-aa8e-49cc-bb70-2cb98c30ad65"
-					(reference "C22")
+					(reference "C901")
 					(unit 1)
 				)
@@
 		(dnp no)
 		(fields_autoplaced yes)
-		(property "Reference" "#PWR033"
+		(property "Reference" "#PWR0901"
 			(at 134.62 116.84 0)
 			(effects
@@
 			(project "cubesat_rp2040"
 				(path "/5511013b-c214-40ba-8960-f470f52474f8/1dd649c8-aa8e-49cc-bb70-2cb98c30ad65"
-					(reference "#PWR033")
+					(reference "#PWR0901")
 					(unit 1)
 				)
@@
 		(dnp no)
 		(fields_autoplaced yes)
-		(property "Reference" "R15"
+		(property "Reference" "R901"
 			(at 143.51 88.9 90)
 			(effects
@@
 			)
 		)
-		(property "Footprint" "Resistor_SMD:R_0402_1005Metric"
+		(property "Footprint" "cubesat_rp2040:R_0402_1005Metric"
 			(at 143.51 93.472 90)
 			(effects
@@
 			(project "cubesat_rp2040"
 				(path "/5511013b-c214-40ba-8960-f470f52474f8/1dd649c8-aa8e-49cc-bb70-2cb98c30ad65"
-					(reference "R15")
+					(reference "R901")
 					(unit 1)
 				)
@@
 		(dnp no)
 		(fields_autoplaced yes)
-		(property "Reference" "#PWR035"
+		(property "Reference" "#PWR0903"
 			(at 157.48 116.84 0)
 			(effects
@@
 			(project "cubesat_rp2040"
 				(path "/5511013b-c214-40ba-8960-f470f52474f8/1dd649c8-aa8e-49cc-bb70-2cb98c30ad65"
-					(reference "#PWR035")
+					(reference "#PWR0903")
 					(unit 1)
 				)
@@
 		(dnp no)
 		(fields_autoplaced yes)
-		(property "Reference" "R16"
+		(property "Reference" "R902"
 			(at 154.94 87.63 0)
 			(effects
@@
 			)
 		)
-		(property "Footprint" "Resistor_SMD:R_0402_1005Metric"
+		(property "Footprint" "cubesat_rp2040:R_0402_1005Metric"
 			(at 150.622 88.9 90)
 			(effects
@@
 			(project "cubesat_rp2040"
 				(path "/5511013b-c214-40ba-8960-f470f52474f8/1dd649c8-aa8e-49cc-bb70-2cb98c30ad65"
-					(reference "R16")
+					(reference "R902")
 					(unit 1)
 				)
@@
 		(dnp no)
 		(fields_autoplaced yes)
-		(property "Reference" "#PWR034"
+		(property "Reference" "#PWR0902"
 			(at 152.4 86.36 0)
 			(effects
@@
 			(project "cubesat_rp2040"
 				(path "/5511013b-c214-40ba-8960-f470f52474f8/1dd649c8-aa8e-49cc-bb70-2cb98c30ad65"
-					(reference "#PWR034")
+					(reference "#PWR0902")
 					(unit 1)
 				)
@@
 		(dnp no)
 		(fields_autoplaced yes)
-		(property "Reference" "SW1"
+		(property "Reference" "SW901"
 			(at 135.89 101.6 90)
 			(effects
@@
 			(project "cubesat_rp2040"
 				(path "/5511013b-c214-40ba-8960-f470f52474f8/1dd649c8-aa8e-49cc-bb70-2cb98c30ad65"
-					(reference "SW1")
+					(reference "SW901")
 					(unit 1)
 				)

Commit message: Major update, everything has been touched
Parts:
- renumbered C901 to C801, R901 to R801, R902 to R802, SW901 to SW801
Changed lines of the file:
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@@
 		(dnp no)
 		(fields_autoplaced yes)
-		(property "Reference" "C901"
+		(property "Reference" "C801"
 			(at 161.29 101.5999 0)
 			(effects
@@
 			(project "cubesat_rp2040"
 				(path "/5511013b-c214-40ba-8960-f470f52474f8/1dd649c8-aa8e-49cc-bb70-2cb98c30ad65"
-					(reference "C901")
+					(reference "C801")
 					(unit 1)
 				)
@@
 		(dnp no)
 		(fields_autoplaced yes)
-		(property "Reference" "#PWR0901"
+		(property "Reference" "#PWR0801"
 			(at 134.62 116.84 0)
 			(effects
@@
 			(project "cubesat_rp2040"
 				(path "/5511013b-c214-40ba-8960-f470f52474f8/1dd649c8-aa8e-49cc-bb70-2cb98c30ad65"
-					(reference "#PWR0901")
+					(reference "#PWR0801")
 					(unit 1)
 				)
@@
 		(dnp no)
 		(fields_autoplaced yes)
-		(property "Reference" "R901"
+		(property "Reference" "R801"
 			(at 143.51 88.9 90)
 			(effects
@@
 			(project "cubesat_rp2040"
 				(path "/5511013b-c214-40ba-8960-f470f52474f8/1dd649c8-aa8e-49cc-bb70-2cb98c30ad65"
-					(reference "R901")
+					(reference "R801")
 					(unit 1)
 				)
@@
 		(dnp no)
 		(fields_autoplaced yes)
-		(property "Reference" "#PWR0903"
+		(property "Reference" "#PWR0803"
 			(at 157.48 116.84 0)
 			(effects
@@
 			(project "cubesat_rp2040"
 				(path "/5511013b-c214-40ba-8960-f470f52474f8/1dd649c8-aa8e-49cc-bb70-2cb98c30ad65"
-					(reference "#PWR0903")
+					(reference "#PWR0803")
 					(unit 1)
 				)
@@
 		(dnp no)
 		(fields_autoplaced yes)
-		(property "Reference" "R902"
+		(property "Reference" "R802"
 			(at 154.94 87.63 0)
 			(effects
@@
 			(project "cubesat_rp2040"
 				(path "/5511013b-c214-40ba-8960-f470f52474f8/1dd649c8-aa8e-49cc-bb70-2cb98c30ad65"
-					(reference "R902")
+					(reference "R802")
 					(unit 1)
 				)
@@
 		(dnp no)
 		(fields_autoplaced yes)
-		(property "Reference" "#PWR0902"
+		(property "Reference" "#PWR0802"
 			(at 152.4 86.36 0)
 			(effects
@@
 			(project "cubesat_rp2040"
 				(path "/5511013b-c214-40ba-8960-f470f52474f8/1dd649c8-aa8e-49cc-bb70-2cb98c30ad65"
-					(reference "#PWR0902")
+					(reference "#PWR0802")
 					(unit 1)
 				)
@@
 		(dnp no)
 		(fields_autoplaced yes)
-		(property "Reference" "SW901"
+		(property "Reference" "SW801"
 			(at 135.89 101.6 90)
 			(effects
@@
 			(project "cubesat_rp2040"
 				(path "/5511013b-c214-40ba-8960-f470f52474f8/1dd649c8-aa8e-49cc-bb70-2cb98c30ad65"
-					(reference "SW901")
-					(unit 1)
-				)
+					(reference "SW801")
+					(unit 1)
+				)
