File: usb.kicad_sch (KiCad schematic)
At the start: 7 parts, among them J301 USB_C_Receptacle_USB2.0

Commit message: Major update, everything has been touched
Parts:
- removed C301: 100n, cubesat_rp2040:C_0402_1005Metric, symbol Device:C
- removed C302: 1n, cubesat_rp2040:C_0402_1005Metric, symbol Device:C
- removed C303: 10u, cubesat_rp2040:C_0402_1005Metric, symbol Device:C
- added C304, C305: 1u, cubesat_rp2040:C_0402_1005Metric, symbol Device:C
- added C306, C307, C308, C309, C310, C311, C312, C313, C314, C315, C316: 100n, cubesat_rp2040:C_0402_1005Metric, symbol Device:C
- added D302, D303: D_TVS, Diode_SMD:D_0402_1005Metric, symbol Device:D_TVS
- added R304: 90.9k 1%, cubesat_rp2040:R_0402_1005Metric, symbol Device:R
- added R306: 9.53k 1%, cubesat_rp2040:R_0402_1005Metric, symbol Device:R
- added R307, R308, R309, R310, R311: 4.7k, cubesat_rp2040:R_0402_1005Metric, symbol Device:R
- added U301: TUSB4041I, Package_QFP:HTQFP-64-1EP_10x10mm_P0.5mm_EP8x8mm_Mask4.4x4.4mm_ThermalVias, symbol cubesat_rp2040:TUSB4041I
- R301: MANUFACTURER (none) -> Vishay; Manufacturer_Name (none) -> Vishay; Manufacturer_Part_Number (none) -> P-0402E5101FGxx
- R303: renamed from R302; MANUFACTURER (none) -> Vishay; Manufacturer_Name (none) -> Vishay; Manufacturer_Part_Number (none) -> P-0402E5101FGxx
- R305: value 1M -> 10k 1%; MANUFACTURER (none) -> Vishay; Manufacturer_Name (none) -> Vishay; Manufacturer_Part_Number (none) -> P-0402E1002FGxx
Connections:
- net GND: now also J301.S1 (SHIELD), C304.2, C305.2, C306.2, C307.2, C308.2, C309.2, C310.2, C311.2, C312.2, C313.2, C314.2, C315.2, C316.2, D302.1 (A1), D303.1 (A1), R306.2, R307.2, R308.2, R309.2, R310.2, R311.2, U301.65 (VSS)
- net USB_UP.D+: now also D302.2 (A2), U301.21 (USB_DP_UP)
- net USB_UP.D-: now also D303.2 (A2), U301.22 (USB_DM_UP)
- net VBUS: now also R304.1
- net Earth renamed USB_VBUS
- net USB_VBUS: now also R304.2, U301.16 (USB_VBUS); no longer J301.S1 (SHIELD)
- new net: R307.1, U301.10 (GANGED/SMBA2/HS_UP)
- new net: R306.1, U301.32 (USB_R1)
- new net +1V1: C304.1, C306.1, C307.1, C308.1, C309.1, C310.1, C311.1, C312.1, U301.19 (VDD), U301.25 (VDD), U301.37 (VDD), U301.45 (VDD), U301.53 (VDD), U301.60 (VDD), U301.63 (VDD)
- new net +3V3: C305.1, C313.1, C314.1, C315.1, C316.1, U301.2 (VDD33), U301.20 (VDD33), U301.31 (VDD33), U301.48 (VDD33)
- new net PWRCTL0/BATEN0: R311.1, U301.4 (PWRCTL1/BATEN1)
- new net PWRCTL1/BATEN1: R310.1, U301.3 (PWRCTL2/BATEN2)
- new net PWRCTL2/BATEN2: R309.1, U301.1 (PWRCTL3/BATEN3)
- new net PWRCTL3/BATEN3: R308.1, U301.64 (PWRCTL4/BATEN4)
- new net USB_DN0.D+: U301.33 (USB_DP_DN1)
- new net USB_DN0.D-: U301.34 (USB_DM_DN1)
- new net USB_DN1.D+: U301.41 (USB_DP_DN2)
- new net USB_DN1.D-: U301.42 (USB_DM_DN2)
- new net USB_DN2.D+: U301.49 (USB_DP_DN3)
- new net USB_DN2.D-: U301.50 (USB_DM_DN3)
- new net USB_DN3.D+: U301.56 (USB_DP_DN4)
- new net USB_DN3.D-: U301.57 (USB_DM_DN4)
- new net XIN: U301.30 (XI)
- new net ~{RESET}: U301.18 (GRSTz)
- no-connect marks 2 -> 12
Other:
- moved on the sheet: J301, R301, R303
