File: usb.kicad_sch (KiCad schematic)
At the start: 27 parts, among them J301 USB_C_Receptacle_USB2.0, U301 TUSB4041I

Commit message: Another large revision, but we are getting closer
Parts:
- C10: renamed from C306; value 100n -> 100nF; LCSC_Part_Number (none) -> C960916; MANUFACTURER (none) -> Samsung Electro-Mechanics; Manufacturer_Name (none) -> Samsung Electro-Mechanics; Manufacturer_Part_Number (none) -> CL05B104KB5NNNC
- C11: renamed from C307; value 100n -> 100nF; LCSC_Part_Number (none) -> C960916; MANUFACTURER (none) -> Samsung Electro-Mechanics; Manufacturer_Name (none) -> Samsung Electro-Mechanics; Manufacturer_Part_Number (none) -> CL05B104KB5NNNC
- C12: renamed from C308; value 100n -> 100nF; LCSC_Part_Number (none) -> C960916; MANUFACTURER (none) -> Samsung Electro-Mechanics; Manufacturer_Name (none) -> Samsung Electro-Mechanics; Manufacturer_Part_Number (none) -> CL05B104KB5NNNC
- C13: renamed from C309; value 100n -> 100nF; LCSC_Part_Number (none) -> C960916; MANUFACTURER (none) -> Samsung Electro-Mechanics; Manufacturer_Name (none) -> Samsung Electro-Mechanics; Manufacturer_Part_Number (none) -> CL05B104KB5NNNC
- C14: renamed from C310; value 100n -> 100nF; LCSC_Part_Number (none) -> C960916; MANUFACTURER (none) -> Samsung Electro-Mechanics; Manufacturer_Name (none) -> Samsung Electro-Mechanics; Manufacturer_Part_Number (none) -> CL05B104KB5NNNC
- C15: renamed from C311; value 100n -> 100nF; LCSC_Part_Number (none) -> C960916; MANUFACTURER (none) -> Samsung Electro-Mechanics; Manufacturer_Name (none) -> Samsung Electro-Mechanics; Manufacturer_Part_Number (none) -> CL05B104KB5NNNC
- C16: renamed from C312; value 100n -> 100nF; LCSC_Part_Number (none) -> C960916; MANUFACTURER (none) -> Samsung Electro-Mechanics; Manufacturer_Name (none) -> Samsung Electro-Mechanics; Manufacturer_Part_Number (none) -> CL05B104KB5NNNC
- C17: renamed from C313; value 100n -> 100nF; LCSC_Part_Number (none) -> C960916; MANUFACTURER (none) -> Samsung Electro-Mechanics; Manufacturer_Name (none) -> Samsung Electro-Mechanics; Manufacturer_Part_Number (none) -> CL05B104KB5NNNC
- C18: renamed from C314; value 100n -> 100nF; LCSC_Part_Number (none) -> C960916; MANUFACTURER (none) -> Samsung Electro-Mechanics; Manufacturer_Name (none) -> Samsung Electro-Mechanics; Manufacturer_Part_Number (none) -> CL05B104KB5NNNC
- C19: renamed from C315; value 100n -> 100nF; LCSC_Part_Number (none) -> C960916; MANUFACTURER (none) -> Samsung Electro-Mechanics; Manufacturer_Name (none) -> Samsung Electro-Mechanics; Manufacturer_Part_Number (none) -> CL05B104KB5NNNC
- C20: renamed from C316; value 100n -> 100nF; LCSC_Part_Number (none) -> C960916; MANUFACTURER (none) -> Samsung Electro-Mechanics; Manufacturer_Name (none) -> Samsung Electro-Mechanics; Manufacturer_Part_Number (none) -> CL05B104KB5NNNC
- C8: renamed from C304; value 1u -> 1uF; footprint cubesat_rp2040:C_0402_1005Metric -> Capacitor_SMD:C_0805_2012Metric; LCSC_Part_Number (none) -> C28323; MANUFACTURER (none) -> Samsung Electro-Mechanics; Manufacturer_Name (none) -> Samsung Electro-Mechanics; Manufacturer_Part_Number (none) -> CL21B105KBFNNNE
- C9: renamed from C305; value 1u -> 1uF; footprint cubesat_rp2040:C_0402_1005Metric -> Capacitor_SMD:C_0805_2012Metric; LCSC_Part_Number (none) -> C28323; MANUFACTURER (none) -> Samsung Electro-Mechanics; Manufacturer_Name (none) -> Samsung Electro-Mechanics; Manufacturer_Part_Number (none) -> CL21B105KBFNNNE
- D14: renamed from D302; LCSC_Part_Number (none) -> C1973257; Manufacturer_Name (none) -> Kyocera AVX; Manufacturer_Part_Number (none) -> GG0402052R542P
- D15: renamed from D303; LCSC_Part_Number (none) -> C1973257; Manufacturer_Name (none) -> Kyocera AVX; Manufacturer_Part_Number (none) -> GG0402052R542P
- J4: renamed from J301; LCSC_Part_Number (none) -> C5299418; Manufacturer_Name (none) -> G-Switch; Manufacturer_Part_Number (none) -> GT-USB-9010ANS
- R11: renamed from R301; value 5.1k 10% -> 5.1kR 10%; LCSC_Part_Number (none) -> C490833; Manufacturer_Name Vishay -> PANASONIC; Manufacturer_Part_Number P-0402E5101FGxx -> ERA2AEB512X
- R12: renamed from R303; value 5.1k 10% -> 5.1kR 10%; LCSC_Part_Number (none) -> C490833; Manufacturer_Name Vishay -> PANASONIC; Manufacturer_Part_Number P-0402E5101FGxx -> ERA2AEB512X
- R13: renamed from R304; value 90.9k 1% -> 90.9kR 1%; LCSC_Part_Number (none) -> C26989; Manufacturer_Name Vishay -> UNI-ROYAL(Uniroyal Elec); Manufacturer_Part_Number P-0402E9092FGxx -> 0402WGF9092TCE
- R14: renamed from R305; value 10k 1% -> 10kR 1%; LCSC_Part_Number (none) -> C191568; Manufacturer_Name Vishay -> PANASONIC; Manufacturer_Part_Number P-0402E1002FGxx -> ERA2AED103X
- R15: renamed from R306; value 9.53k 1% -> 9.53kR 1%; LCSC_Part_Number (none) -> C96273; Manufacturer_Name Vishay -> UNI-ROYAL(Uniroyal Elec); Manufacturer_Part_Number P-0402E9531FGxx -> 0402WGF9531TCE
- R16: renamed from R307; value 4.7k -> 4.7kR; LCSC_Part_Number (none) -> C490830; Manufacturer_Name Vishay -> PANASONIC; Manufacturer_Part_Number P-0402E4701FGxx -> ERA2AEB472X
- R17: renamed from R308; value 4.7k -> 4.7kR; LCSC_Part_Number (none) -> C490830; Manufacturer_Name Vishay -> PANASONIC; Manufacturer_Part_Number P-0402E4701FGxx -> ERA2AEB472X
- R18: renamed from R309; value 4.7k -> 4.7kR; LCSC_Part_Number (none) -> C490830; Manufacturer_Name Vishay -> PANASONIC; Manufacturer_Part_Number P-0402E4701FGxx -> ERA2AEB472X
- R19: renamed from R310; value 4.7k -> 4.7kR; LCSC_Part_Number (none) -> C490830; Manufacturer_Name Vishay -> PANASONIC; Manufacturer_Part_Number P-0402E4701FGxx -> ERA2AEB472X
- R20: renamed from R311; value 4.7k -> 4.7kR; LCSC_Part_Number (none) -> C490830; Manufacturer_Name Vishay -> PANASONIC; Manufacturer_Part_Number P-0402E4701FGxx -> ERA2AEB472X
- U2: renamed from U301; footprint Package_QFP:HTQFP-64-1EP_10x10mm_P0.5mm_EP8x8mm_Mask4.4x4.4mm_ThermalVias -> cubesat_rp2040:HTQFP-64-1EP_10x10mm_P0.5mm_EP8x8mm_Mask4.4x4.4mm_ThermalVias; LCSC_Part_Number (none) -> C702377; Manufacturer_Name (none) -> Texas Instruments; Manufacturer_Part_Number (none) -> TUSB4041IPAPRQ1
Connections:
- net PWRCTL0/BATEN0 is gone; now on net PWRCTL1/BATEN1: R20.1, U2.4 (PWRCTL1/BATEN1)
- net USB_DN0.D+ is gone; now on net USB_DN1.D+: U2.33 (USB_DP_DN1)
- net USB_DN0.D- is gone; now on net USB_DN1.D-: U2.34 (USB_DM_DN1)
- net PWRCTL1/BATEN1: no longer R19.1, U2.3 (PWRCTL2/BATEN2)
- net PWRCTL2/BATEN2: now also R19.1, U2.3 (PWRCTL2/BATEN2); no longer R18.1, U2.1 (PWRCTL3/BATEN3)
- net PWRCTL3/BATEN3: now also R18.1, U2.1 (PWRCTL3/BATEN3); no longer R17.1, U2.64 (PWRCTL4/BATEN4)
- net USB_DN1.D+: no longer U2.41 (USB_DP_DN2)
- net USB_DN1.D-: no longer U2.42 (USB_DM_DN2)
- net USB_DN2.D+: now also U2.41 (USB_DP_DN2); no longer U2.49 (USB_DP_DN3)
- net USB_DN2.D-: now also U2.42 (USB_DM_DN2); no longer U2.50 (USB_DM_DN3)
- net USB_DN3.D+: now also U2.49 (USB_DP_DN3); no longer U2.56 (USB_DP_DN4)
- net USB_DN3.D-: now also U2.50 (USB_DM_DN3); no longer U2.57 (USB_DM_DN4)
- net XIN renamed CLK_24MHz
- new net PWRCTL4/BATEN4: R17.1, U2.64 (PWRCTL4/BATEN4)
- new net USB_DN4.D+: U2.56 (USB_DP_DN4)
- new net USB_DN4.D-: U2.57 (USB_DM_DN4)

Commit message: More work on interfaces
Parts:
- added R9: 4.7kR, cubesat_rp2040:R_0402_1005Metric, symbol Device:R
- renumbered C16 to C10, C17 to C11, C18 to C12, C19 to C13, C20 to C14, C8 to C2, C9 to C3, C10 to C4, C11 to C5, C12 to C6, C13 to C7, C14 to C8, C15 to C9, D14 to D13, D15 to D14, R17 to R10, R18 to R11, R19 to R12, R20 to R13, R11 to R3, R12 to R4, R13 to R5, R16 to R6, R14 to R7, R15 to R8, U2 to U1
Connections:
- net GND: now also R9.2
- net at U1.13 (AUTOENz/HS_SUSPEND): now also R9.1
- no-connect marks 12 -> 13
Other:
- moved on the sheet: R6
