File: L7983_5V_stepdown_3V3.kicad_sch (KiCad schematic)
At the start: 13 parts, among them U201 L7983

Commit message: Major update, everything has been touched
Parts:
- removed R206: R, symbol Device:R
- added C203: 470n, cubesat_rp2040:C_0402_1005Metric, symbol Device:C
- added C206: 10u, Capacitor_SMD:C_0805_2012Metric, symbol Device:C
- added R203: 100k, cubesat_rp2040:R_0402_1005Metric, symbol Device:R
- added R204: 56k, cubesat_rp2040:R_0402_1005Metric, symbol Device:R
- added R208: 470R, cubesat_rp2040:R_0402_1005Metric, symbol Device:R
- C201: renamed from C202; footprint cubesat_rp2040:C_0402_1005Metric -> Capacitor_SMD:C_0805_2012Metric
- C205: renamed from C204; footprint cubesat_rp2040:C_0402_1005Metric -> Capacitor_SMD:C_0805_2012Metric
- D201: value LED -> GREEN; footprint (none) -> LED_SMD:LED_0402_1005Metric
- R201: MANUFACTURER (none) -> Vishay; Manufacturer_Name (none) -> Vishay; Manufacturer_Part_Number (none) -> P-0402E5602FGxx
- R202: MANUFACTURER (none) -> Vishay; Manufacturer_Name (none) -> Vishay; Manufacturer_Part_Number (none) -> P-0402E4702FGxx
- R205: renamed from R203; MANUFACTURER (none) -> Vishay; Manufacturer_Name (none) -> Vishay; Manufacturer_Part_Number (none) -> P-0402E1003FGxx
- R206: renamed from R204; MANUFACTURER (none) -> Vishay; Manufacturer_Name (none) -> Vishay; Manufacturer_Part_Number (none) -> P-0402E4702FGxx
- R207: renamed from R205; MANUFACTURER (none) -> Vishay; Manufacturer_Name (none) -> Vishay; Manufacturer_Part_Number (none) -> P-0402E1602FGxx
- renumbered C201 to C202, C203 to C204
Connections:
- net GND: now also D201.1 (K), C203.2, C206.2, R204.1
- net VIN: now also R203.2; no longer U201.7 (EN/UVLO)
- net ~{RESET}: now also R208.1
- net FB: now reaches R206.2, R207.1, U201.1 (VOUT/FB)
- net LX: now reaches L201.1, U201.9 (LX)
- net at D201.2 (A): now also R208.2
- new net EN/UVLO: C203.1, R203.1, R204.2, U201.7 (EN/UVLO)
- new net VBUS: C206.1
Other:
- moved on the sheet: C201, C202, C204, C205, L201, R201, R202, R205, R206, R207, U201

Commit message: Another large revision, but we are getting closer
Parts:
- C2: renamed from C201; value 1u -> 1uF; LCSC_Part_Number (none) -> C28323; Manufacturer_Name (none) -> Samsung Electro-Mechanics; Manufacturer_Part_Number (none) -> CL21B105KBFNNNE
- C3: renamed from C202; value 470n -> 470nF; footprint cubesat_rp2040:C_0402_1005Metric -> Capacitor_SMD:C_0805_2012Metric; LCSC_Part_Number (none) -> C13967; MANUFACTURER (none) -> Samsung Electro-Mechanics; Manufacturer_Name (none) -> Samsung Electro-Mechanics; Manufacturer_Part_Number (none) -> CL21B474KBFNNNE
- C4: renamed from C203; value 470n -> 470nF; footprint cubesat_rp2040:C_0402_1005Metric -> Capacitor_SMD:C_0805_2012Metric; LCSC_Part_Number (none) -> C13967; MANUFACTURER (none) -> Samsung Electro-Mechanics; Manufacturer_Name (none) -> Samsung Electro-Mechanics; Manufacturer_Part_Number (none) -> CL21B474KBFNNNE
- C5: renamed from C204; value 100n -> 100nF; LCSC_Part_Number (none) -> C960916; MANUFACTURER (none) -> Samsung Electro-Mechanics; Manufacturer_Name (none) -> Samsung Electro-Mechanics; Manufacturer_Part_Number (none) -> CL05B104KB5NNNC
- C6: renamed from C205; value 1u -> 1uF; LCSC_Part_Number (none) -> C28323; Manufacturer_Name (none) -> Samsung Electro-Mechanics; Manufacturer_Part_Number (none) -> CL21B105KBFNNNE
- C7: renamed from C206; value 10u -> 10uF; footprint Capacitor_SMD:C_0805_2012Metric -> Capacitor_SMD:C_1206_3216Metric; LCSC_Part_Number (none) -> C89632; Manufacturer_Name (none) -> Samsung Electro-Mechanics; Manufacturer_Part_Number (none) -> CL31B106KBHNNNE
- D13: renamed from D201; LCSC_Part_Number (none) -> C364551; Manufacturer_Name (none) -> Lite-On; Manufacturer_Part_Number (none) -> LTST-C281KGKT-5A
- L1: renamed from L201; value 10u -> 10uH; LCSC_Part_Number (none) -> C2047632; Manufacturer_Name (none) -> TDK; Manufacturer_Part_Number (none) -> TFM322512ALMA100MTAA
- R10: renamed from R208; LCSC_Part_Number (none) -> C445590; Manufacturer_Name Vishay -> PANASONIC; Manufacturer_Part_Number P-0402E4700FGxx -> ERA2AEB471X
- R3: renamed from R201; value 56k -> 56kR; LCSC_Part_Number (none) -> C445617; Manufacturer_Name Vishay -> PANASONIC; Manufacturer_Part_Number P-0402E5602FGxx -> ERA2AEB563X
- R4: renamed from R202; value 47k -> 47kR; LCSC_Part_Number (none) -> C543615; Manufacturer_Name Vishay -> PANASONIC; Manufacturer_Part_Number P-0402E4702FGxx -> ERA2AEB473X
- R5: renamed from R203; value 100k -> 100kR; LCSC_Part_Number (none) -> C191569; Manufacturer_Name Vishay -> PANASONIC; Manufacturer_Part_Number P-0402E1003FGxx -> ERA2AED104X
- R6: renamed from R204; value 56k -> 56kR; LCSC_Part_Number (none) -> C445617; Manufacturer_Name Vishay -> PANASONIC; Manufacturer_Part_Number P-0402E5602FGxx -> ERA2AEB563X
- R7: renamed from R205; value 100k -> 100kR; LCSC_Part_Number (none) -> C191569; Manufacturer_Name Vishay -> PANASONIC; Manufacturer_Part_Number P-0402E1003FGxx -> ERA2AED104X
- R8: renamed from R206; value 47k -> 47kR; LCSC_Part_Number (none) -> C543615; Manufacturer_Name Vishay -> PANASONIC; Manufacturer_Part_Number P-0402E4702FGxx -> ERA2AEB473X
- R9: renamed from R207; value 16k -> 16kR; LCSC_Part_Number (none) -> C543609; Manufacturer_Name Vishay -> PANASONIC; Manufacturer_Part_Number P-0402E1602FGxx -> ERA2AEB163X
- renumbered U201 to U1
Connections:
- net GND: now also R10.1; no longer D13.1 (K)
- net ~{RESET}: now also D13.2 (A); no longer R10.1
- net at R10.2: now also D13.1 (K); no longer D13.2 (A)
Other:
- moved on the sheet: D13, R10
