File: RST3225N_TCXO_32M0.kicad_sch (KiCad schematic)
At the start: 5 parts, among them U801 RST3225N

Commit message: Big update, bad commit messsage :)
Parts:
- C803, C804: footprint Capacitor_SMD:C_0402_1005Metric -> cubesat_rp2040:C_0402_1005Metric
- R802, R803: footprint Resistor_SMD:R_0402_1005Metric -> cubesat_rp2040:R_0402_1005Metric
- U801: value RST3225N -> T6405 R24M0
Other:
- title: RST3225N TCXO -> CubeSat RP2040 Board
- moved on the sheet: C803, R802
Changed lines of the file:
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@@
 	(paper "A4")
 	(title_block
-		(title "RST3225N TCXO")
+		(title "CubeSat RP2040 Board")
 		(rev "1")
 		(company "Magnus Oksbøl Therkelsen")
+		(comment 1 "Author: Magnus Oksbøl Therkelsen")
+		(comment 2 "Checked by: ")
 	)
 	(junction
@@
 	)
 	(junction
-		(at 127 88.9)
+		(at 114.3 88.9)
+		(diameter 0)
+		(color 0 0 0 0)
+	)
+	(junction
+		(at 152.4 88.9)
 		(diameter 0)
 		(color 0 0 0 0)
@@
 	(wire
 		(pts
-			(xy 127 88.9) (xy 152.4 88.9)
+			(xy 88.9 76.2) (xy 88.9 88.9)
+		)
+		(stroke
+			(width 0)
+			(type default)
+		)
+	)
+	(wire
+		(pts
+			(xy 114.3 88.9) (xy 152.4 88.9)
 		)
 		(stroke
@@
 	(wire
 		(pts
+			(xy 152.4 86.36) (xy 152.4 88.9)
+		)
+		(stroke
+			(width 0)
+			(type default)
+		)
+	)
+	(wire
+		(pts
 			(xy 177.8 111.76) (xy 177.8 120.65)
 		)
@@
 	(wire
 		(pts
-			(xy 127 88.9) (xy 127 97.79)
+			(xy 114.3 88.9) (xy 114.3 97.79)
 		)
 		(stroke
@@
 	(wire
 		(pts
-			(xy 118.11 88.9) (xy 127 88.9)
-		)
-		(stroke
-			(width 0)
-			(type default)
-		)
-	)
-	(wire
-		(pts
-			(xy 101.6 76.2) (xy 101.6 88.9)
-		)
-		(stroke
-			(width 0)
-			(type default)
-		)
-	)
-	(wire
-		(pts
-			(xy 101.6 88.9) (xy 110.49 88.9)
-		)
-		(stroke
-			(width 0)
-			(type default)
-		)
-	)
-	(wire
-		(pts
-			(xy 127 105.41) (xy 127 120.65)
+			(xy 105.41 88.9) (xy 114.3 88.9)
+		)
+		(stroke
+			(width 0)
+			(type default)
+		)
+	)
+	(wire
+		(pts
+			(xy 88.9 88.9) (xy 97.79 88.9)
+		)
+		(stroke
+			(width 0)
+			(type default)
+		)
+	)
+	(wire
+		(pts
+			(xy 114.3 105.41) (xy 114.3 120.65)
 		)
 		(stroke
@@
 			)
 		)
-		(property "Footprint" "Capacitor_SMD:C_0402_1005Metric"
+		(property "Footprint" "cubesat_rp2040:C_0402_1005Metric"
 			(at 175.26 100.6348 0)
 			(effects
@@
 			)
 		)
-		(property "Value" "RST3225N"
+		(property "Value" "T6405 R24M0"
 			(at 144.78 102.8699 0)
 			(effects
@@
 	(symbol
 		(lib_id "power:+3V3")
-		(at 101.6 76.2 0)
+		(at 88.9 76.2 0)
 		(unit 1)
 		(exclude_from_sim no)
@@
 		(fields_autoplaced yes)
 		(property "Reference" "#PWR0802"
-			(at 101.6 80.01 0)
+			(at 88.9 80.01 0)
 			(effects
 				(font
@@
 		)
 		(property "Value" "+3V3"
-			(at 101.6 71.12 0)
+			(at 88.9 71.12 0)
 			(effects
 				(font
@@
 		)
 		(property "Footprint" ""
-			(at 101.6 76.2 0)
+			(at 88.9 76.2 0)
 			(effects
 				(font
@@
 		)
 		(property "Datasheet" ""
-			(at 101.6 76.2 0)
+			(at 88.9 76.2 0)
 			(effects
 				(font
@@
 		)
 		(property "Description" "Power symbol creates a global label with name \"+3V3\""
-			(at 101.6 76.2 0)
+			(at 88.9 76.2 0)
 			(effects
 				(font
@@
 	(symbol
 		(lib_id "Device:R")
-		(at 114.3 88.9 90)
+		(at 101.6 88.9 90)
 		(unit 1)
 		(exclude_from_sim no)
@@
 		(fields_autoplaced yes)
 		(property "Reference" "R802"
-			(at 114.3 82.55 90)
+			(at 101.6 82.55 90)
 			(effects
 				(font
@@
 		)
 		(property "Value" "33R"
-			(at 114.3 85.09 90)
-			(effects
-				(font
-					(size 1.27 1.27)
-				)
-			)
-		)
-		(property "Footprint" "Resistor_SMD:R_0402_1005Metric"
-			(at 114.3 90.678 90)
+			(at 101.6 85.09 90)
+			(effects
+				(font
+					(size 1.27 1.27)
+				)
+			)
+		)
+		(property "Footprint" "cubesat_rp2040:R_0402_1005Metric"
+			(at 101.6 90.678 90)
 			(effects
 				(font
@@
 		)
 		(property "Datasheet" "~"
-			(at 114.3 88.9 0)
+			(at 101.6 88.9 0)
 			(effects
 				(font
@@
 		)
 		(property "Description" "Resistor"
-			(at 114.3 88.9 0)
+			(at 101.6 88.9 0)
 			(effects
 				(font
@@
 	(symbol
 		(lib_id "power:GND")
-		(at 127 120.65 0)
+		(at 114.3 120.65 0)
 		(unit 1)
 		(exclude_from_sim no)
@@
 		(fields_autoplaced yes)
 		(property "Reference" "#PWR0804"
-			(at 127 127 0)
+			(at 114.3 127 0)
 			(effects
 				(font
@@
 		)
 		(property "Value" "GND"
-			(at 127 125.73 0)
+			(at 114.3 125.73 0)
 			(effects
 				(font
@@
 		)
 		(property "Footprint" ""
-			(at 127 120.65 0)
+			(at 114.3 120.65 0)
 			(effects
 				(font
@@
 		)
 		(property "Datasheet" ""
-			(at 127 120.65 0)
+			(at 114.3 120.65 0)
 			(effects
 				(font
@@
 		)
 		(property "Description" "Power symbol creates a global label with name \"GND\" , ground"
-			(at 127 120.65 0)
+			(at 114.3 120.65 0)
 			(effects
 				(font
@@
 	(symbol
 		(lib_id "Device:C")
-		(at 127 101.6 0)
+		(at 114.3 101.6 0)
 		(unit 1)
 		(exclude_from_sim no)
@@
 		(fields_autoplaced yes)
 		(property "Reference" "C803"
-			(at 123.19 100.3299 0)
+			(at 110.49 100.3299 0)
 			(effects
 				(font
@@
 		)
 		(property "Value" "100n"
-			(at 123.19 102.8699 0)
+			(at 110.49 102.8699 0)
 			(effects
 				(font
@@
 			)
 		)
-		(property "Footprint" "Capacitor_SMD:C_0402_1005Metric"
-			(at 127.9652 105.41 0)
+		(property "Footprint" "cubesat_rp2040:C_0402_1005Metric"
+			(at 115.2652 105.41 0)
 			(effects
 				(font
@@
 		)
 		(property "Datasheet" "~"
-			(at 127 101.6 0)
+			(at 114.3 101.6 0)
 			(effects
 				(font
@@
 		)
 		(property "Description" "Unpolarized capacitor"
-			(at 127 101.6 0)
+			(at 114.3 101.6 0)
 			(effects
 				(font
@@
 	)
 	(symbol
+		(lib_id "power:PWR_FLAG")
+		(at 152.4 86.36 0)
+		(unit 1)
+		(exclude_from_sim no)
+		(in_bom yes)
+		(on_board yes)
+		(dnp no)
+		(fields_autoplaced yes)
+		(property "Reference" "#FLG0801"
+			(at 152.4 84.455 0)
+			(effects
+				(font
+					(size 1.27 1.27)
+				)
+				(hide yes)
+			)
+		)
+		(property "Value" "PWR_FLAG"
+			(at 152.4 81.28 0)
+			(effects
+				(font
+					(size 1.27 1.27)
+				)
+			)
+		)
+		(property "Footprint" ""
+			(at 152.4 86.36 0)
+			(effects
+				(font
+					(size 1.27 1.27)
+				)
+				(hide yes)
+			)
+		)
+		(property "Datasheet" "~"
+			(at 152.4 86.36 0)
+			(effects
+				(font
+					(size 1.27 1.27)
+				)
+				(hide yes)
+			)
+		)
+		(property "Description" "Special symbol for telling ERC where power comes from"
+			(at 152.4 86.36 0)
+			(effects
+				(font
+					(size 1.27 1.27)
+				)
+				(hide yes)
+			)
+		)
+		(pin "1"
+		)
+		(instances
+			(project "cubesat_rp2040"
+				(path "/5511013b-c214-40ba-8960-f470f52474f8/9f508e75-6f97-47bb-8ac1-2b188f21985e"
+					(reference "#FLG0801")
+					(unit 1)
+				)
+			)
+		)
+	)
+	(symbol
 		(lib_id "Device:R")
 		(at 177.8 107.95 0)
@@
 			)
 		)
-		(property "Footprint" "Resistor_SMD:R_0402_1005Metric"
+		(property "Footprint" "cubesat_rp2040:R_0402_1005Metric"
 			(at 176.022 107.95 90)
 			(effects

Commit message: Major update, everything has been touched
Parts:
- R401: renamed from R802; MANUFACTURER (none) -> Vishay; Manufacturer_Name (none) -> Vishay; Manufacturer_Part_Number (none) -> P-0402E33R0FGxx
- R402: renamed from R803; MANUFACTURER (none) -> Vishay; Manufacturer_Name (none) -> Vishay; Manufacturer_Part_Number (none) -> P-0402E1002FGxx
- renumbered C803 to C401, C804 to C402, U801 to U401
Changed lines of the file:
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@@
 	(generator "eeschema")
 	(generator_version "8.0")
-	(paper "A4")
+	(paper "A3")
 	(title_block
 		(title "CubeSat RP2040 Board")
@@
 		(dnp no)
 		(fields_autoplaced yes)
-		(property "Reference" "C804"
+		(property "Reference" "C402"
 			(at 171.45 93.98 90)
 			(effects
@@
 			(project "cubesat_rp2040"
 				(path "/5511013b-c214-40ba-8960-f470f52474f8/9f508e75-6f97-47bb-8ac1-2b188f21985e"
-					(reference "C804")
+					(reference "C402")
 					(unit 1)
 				)
@@
 		(dnp no)
 		(fields_autoplaced yes)
-		(property "Reference" "#PWR0805"
+		(property "Reference" "#PWR0404"
 			(at 177.8 127 0)
 			(effects
@@
 			(project "cubesat_rp2040"
 				(path "/5511013b-c214-40ba-8960-f470f52474f8/9f508e75-6f97-47bb-8ac1-2b188f21985e"
-					(reference "#PWR0805")
+					(reference "#PWR0404")
 					(unit 1)
 				)
@@
 		(dnp no)
 		(fields_autoplaced yes)
-		(property "Reference" "U801"
+		(property "Reference" "U401"
 			(at 144.78 100.3299 0)
 			(effects
@@
 			(project "cubesat_rp2040"
 				(path "/5511013b-c214-40ba-8960-f470f52474f8/9f508e75-6f97-47bb-8ac1-2b188f21985e"
-					(reference "U801")
+					(reference "U401")
 					(unit 1)
 				)
@@
 		(dnp no)
 		(fields_autoplaced yes)
-		(property "Reference" "#PWR0803"
+		(property "Reference" "#PWR0403"
 			(at 152.4 127 0)
 			(effects
@@
 			(project "cubesat_rp2040"
 				(path "/5511013b-c214-40ba-8960-f470f52474f8/9f508e75-6f97-47bb-8ac1-2b188f21985e"
-					(reference "#PWR0803")
+					(reference "#PWR0403")
 					(unit 1)
 				)
@@
 		(dnp no)
 		(fields_autoplaced yes)
-		(property "Reference" "#PWR0802"
+		(property "Reference" "#PWR0401"
 			(at 88.9 80.01 0)
 			(effects
@@
 			(project "cubesat_rp2040"
 				(path "/5511013b-c214-40ba-8960-f470f52474f8/9f508e75-6f97-47bb-8ac1-2b188f21985e"
-					(reference "#PWR0802")
+					(reference "#PWR0401")
 					(unit 1)
 				)
@@
 		(dnp no)
 		(fields_autoplaced yes)
-		(property "Reference" "R802"
+		(property "Reference" "R401"
 			(at 101.6 82.55 90)
 			(effects
@@
 		)
 		(property "Description" "Resistor"
+			(at 101.6 88.9 0)
+			(effects
+				(font
+					(size 1.27 1.27)
+				)
+				(hide yes)
+			)
+		)
+		(property "MANUFACTURER" "Vishay"
+			(at 101.6 88.9 0)
+			(effects
+				(font
+					(size 1.27 1.27)
+				)
+				(hide yes)
+			)
+		)
+		(property "Manufacturer_Name" "Vishay"
+			(at 101.6 88.9 0)
+			(effects
+				(font
+					(size 1.27 1.27)
+				)
+				(hide yes)
+			)
+		)
+		(property "Manufacturer_Part_Number" "P-0402E33R0FGxx"
 			(at 101.6 88.9 0)
 			(effects
@@
 			(project "cubesat_rp2040"
 				(path "/5511013b-c214-40ba-8960-f470f52474f8/9f508e75-6f97-47bb-8ac1-2b188f21985e"
-					(reference "R802")
+					(reference "R401")
 					(unit 1)
 				)
@@
 		(dnp no)
 		(fields_autoplaced yes)
-		(property "Reference" "#PWR0804"
+		(property "Reference" "#PWR0402"
 			(at 114.3 127 0)
 			(effects
@@
 			(project "cubesat_rp2040"
 				(path "/5511013b-c214-40ba-8960-f470f52474f8/9f508e75-6f97-47bb-8ac1-2b188f21985e"
-					(reference "#PWR0804")
+					(reference "#PWR0402")
 					(unit 1)
 				)
@@
 		(dnp no)
 		(fields_autoplaced yes)
-		(property "Reference" "C803"
+		(property "Reference" "C401"
 			(at 110.49 100.3299 0)
 			(effects
@@
 			(project "cubesat_rp2040"
 				(path "/5511013b-c214-40ba-8960-f470f52474f8/9f508e75-6f97-47bb-8ac1-2b188f21985e"
-					(reference "C803")
+					(reference "C401")
 					(unit 1)
 				)
@@
 		(dnp no)
 		(fields_autoplaced yes)
-		(property "Reference" "#FLG0801"
+		(property "Reference" "#FLG0401"
 			(at 152.4 84.455 0)
 			(effects
@@
 			(project "cubesat_rp2040"
 				(path "/5511013b-c214-40ba-8960-f470f52474f8/9f508e75-6f97-47bb-8ac1-2b188f21985e"
-					(reference "#FLG0801")
+					(reference "#FLG0401")
 					(unit 1)
 				)
@@
 		(dnp no)
 		(fields_autoplaced yes)
-		(property "Reference" "R803"
+		(property "Reference" "R402"
 			(at 180.34 106.6799 0)
 			(effects
@@
 		)
 		(property "Description" "Resistor"
+			(at 177.8 107.95 0)
+			(effects
+				(font
+					(size 1.27 1.27)
+				)
+				(hide yes)
+			)
+		)
+		(property "MANUFACTURER" "Vishay"
+			(at 177.8 107.95 0)
+			(effects
+				(font
+					(size 1.27 1.27)
+				)
+				(hide yes)
+			)
+		)
+		(property "Manufacturer_Name" "Vishay"
+			(at 177.8 107.95 0)
+			(effects
+				(font
+					(size 1.27 1.27)
+				)
+				(hide yes)
+			)
+		)
+		(property "Manufacturer_Part_Number" "P-0402E1002FGxx"
 			(at 177.8 107.95 0)
 			(effects
@@
 			(project "cubesat_rp2040"
 				(path "/5511013b-c214-40ba-8960-f470f52474f8/9f508e75-6f97-47bb-8ac1-2b188f21985e"
-					(reference "R803")
+					(reference "R402")
 					(unit 1)
 				)

Commit message: Another large revision, but we are getting closer
Parts:
- removed U401: T6405 R24M0, cubesat_rp2040:Crystal_SMD_Rakon_3225-4Pin_3.2x2.5mm, symbol cubesat_rp2040:RST3225N
- added C23: 15pF, cubesat_rp2040:C_0402_1005Metric, symbol Device:C
- added X1: YSO140TC, cubesat_rp2040:Oscillator_SMD_YXC_YSO140TC_4Pin_3.2x2.5mm, symbol cubesat_rp2040:YSO140TC
- C21: renamed from C401; value 100n -> 100nF; LCSC_Part_Number (none) -> C960916; MANUFACTURER (none) -> Samsung Electro-Mechanics; Manufacturer_Name (none) -> Samsung Electro-Mechanics; Manufacturer_Part_Number (none) -> CL05B104KB5NNNC
- C22: renamed from C402; value 10n -> 100nF; LCSC_Part_Number (none) -> C960916; MANUFACTURER (none) -> Samsung Electro-Mechanics; Manufacturer_Name (none) -> Samsung Electro-Mechanics; Manufacturer_Part_Number (none) -> CL05B104KB5NNNC
- R21: renamed from R401; LCSC_Part_Number (none) -> C25161; Manufacturer_Name Vishay -> UNI-ROYAL(Uniroyal Elec); Manufacturer_Part_Number P-0402E33R0FGxx -> 0402WGJ0330TCE
- R22: renamed from R402; value 10k -> 88.7R; LCSC_Part_Number (none) -> C423126; Manufacturer_Name Vishay -> UNI-ROYAL(Uniroyal Elec); Manufacturer_Part_Number P-0402E1002FGxx -> 0402WGF887JTCE
Connections:
- net GND: now also C23.1, X1.2 (GND); no longer R22.2
- net at C22.1: now also X1.3 (OUT)
- net at C21.1, R21.2: now also X1.4 (Vdd)
- net F_{out}: no longer names the net of C22.2, R22.1
- new net 24M0_CLK: C23.2, R22.2
- no-connect marks 0 -> 1
Other:
- moved on the sheet: C21, C22, R21, R22
