File: can_phy_unterminated.kicad_sch (KiCad schematic)
At the start: 9 parts, among them U17 TCAN1048AV-Q1

Commit message: More work on interfaces
Parts:
- C91: renamed from C97; now not fitted
- C92: renamed from C98; now not fitted
- R48: renamed from R55; now not fitted
- R49: renamed from R56; now not fitted
- R50: renamed from R57; now not fitted
- R51: renamed from R58; now not fitted
- renumbered C95 to C89, C96 to C90, U17 to U16
Connections:
- net GND: now also U16.15 (EP)
Other:
- title: CubeSat RP2040 Board -> CAN PHY - NO TERMINATION
- moved on the sheet: C89, C90, U16
