File: cubesat_rp2040.kicad_sch (KiCad schematic)
At the start: 23 parts, among them J1 Conn_01x02, J2 ESQ-126-39-G-D, J3 ESQ-126-39-G-D, SW1 SW_Push

Commit message: Clean up project
Other:
- sheet TMR voting renamed TMR
- sheet Oscillator: file RST3225N_TCXO_32M0.kicad_sch -> oscillator.kicad_sch
- sheet TMR: file tmr_voting.kicad_sch -> tmr.kicad_sch
Changed lines of the file:
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@@
 			)
 		)
-		(property "Sheetfile" "RST3225N_TCXO_32M0.kicad_sch"
+		(property "Sheetfile" "oscillator.kicad_sch"
 			(at 25.4 71.7046 0)
 			(effects
@@
 			(color 0 0 0 0.0000)
 		)
-		(property "Sheetname" "TMR voting"
+		(property "Sheetname" "TMR"
 			(at 200.66 57.7084 0)
 			(effects
@@
 			)
 		)
-		(property "Sheetfile" "tmr_voting.kicad_sch"
+		(property "Sheetfile" "tmr.kicad_sch"
 			(at 200.66 84.4046 0)
 			(effects

Commit message: More work on interfaces
Parts:
- removed D1, D10, D11, D12, D2, D3, D4, D5, D6, D7, D8, D9: D_TVS, Diode_SMD:D_0402_1005Metric, symbol Device:D_TVS
- removed J2, J3: ESQ-126-39-G-D, cubesat_rp2040:SAMTEC_ESQ-126-39-G-D_CUBESAT, symbol cubesat_rp2040:ESQ-126-39-G-D
Connections:
- net ~{USB_BOOT} renamed BOOTSEL
- no-connect marks 84 -> 16
Other:
- sheet LVDS renamed M-LVDS PHY
- sheet USB renamed USB PHY
- added sheet CAN PHY - UNIT A (can_phy_unterminated.kicad_sch)
- added sheet CAN PHY - UNIT B (can_phy_unterminated.kicad_sch)
- added sheet CAN PHY - UNIT C (can_phy_terminated.kicad_sch)
- added sheet Cubesat System Bus (cubesat_system_bus.kicad_sch)
- added sheet RS-485 PHY (rs485.kicad_sch)
- sheet M-LVDS PHY ports: added +3V3; removed none
- sheet RP2040 - Unit A ports: added CAN_A{TXD RXD ~{STB}}, CAN_B{TXD RXD ~{STB}}, FLASH_BOOT/~{USB_BOOT}, TMR_VOTE_1, TMR_VOTE_2, VIN, ~{TMR_RESET}, ~{USR_RESET}; removed CAN_A{P N}, CAN_B{P N}, VOTE_1, VOTE_2, ~{USB_BOOT}
- sheet RP2040 - Unit B ports: added CAN_A{TXD RXD ~{STB}}, CAN_B{TXD RXD ~{STB}}, FLASH_BOOT/~{USB_BOOT}, TMR_VOTE_1, TMR_VOTE_2, VIN, ~{TMR_RESET}, ~{USR_RESET}; removed CAN_A{P N}, CAN_B{P N}, VOTE_1, VOTE_2, ~{USB_BOOT}
- sheet RP2040 - Unit C ports: added CAN_A{TXD RXD ~{STB}}, CAN_B{TXD RXD ~{STB}}, FLASH_BOOT/~{USB_BOOT}, TMR_VOTE_1, TMR_VOTE_2, VIN, ~{TMR_RESET}, ~{USR_RESET}; removed CAN_A{P N}, CAN_B{P N}, VOTE_1, VOTE_2, ~{USB_BOOT}
- sheet TMR ports: added {~{TMR_RESET_A} ~{TMR_RESET_B} ~{TMR_RESET_C}}; removed TMR_RESET_A, TMR_RESET_B, TMR_RESET_C
- moved on the sheet: H1, H2, H3, H4
