File: lvds.kicad_sch (KiCad schematic)
At the start: 14 parts, among them U21 SN65LVDS1DBV, U22 SN65LVDS2DBV, U23 SN65LVDS2DBV, U24 SN65LVDS1DBV

Commit message: More work on interfaces
Parts:
- added NT1: NetTie_2, symbol Device:NetTie_2
- renumbered C103 to C100, C104 to C101, C105 to C102, C106 to C103, C99 to C96, C100 to C97, C101 to C98, C102 to C99, R62 to R55, R63 to R56, U21 to U20, U24 to U21
Connections:
- net +3V3_UNIT: now also NT1.2
- net LVDS_TX_B.N: no longer U20.3 (Z)
- new net +3V3: NT1.1
- new net LVDS_TX_A.N: U20.3 (Z)
Other:
- moved on the sheet: C100, C101, C102, C103, C96, C97, C98, C99
