File: oscillator.kicad_sch (KiCad schematic)
At the start: 6 parts, among them X1 YSO140TC

Commit message: More work on interfaces
Parts:
- renumbered C21 to C15, C22 to C16, C23 to C17, R21 to R14, R22 to R15
Changed lines of the file:
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@@
 		(dnp no)
 		(fields_autoplaced yes)
-		(property "Reference" "C22"
+		(property "Reference" "C16"
 			(at 177.8 93.98 90)
 			(effects
@@
 			(project "cubesat_rp2040"
 				(path "/5511013b-c214-40ba-8960-f470f52474f8/9f508e75-6f97-47bb-8ac1-2b188f21985e"
-					(reference "C22")
+					(reference "C16")
 					(unit 1)
 				)
@@
 		(dnp no)
 		(fields_autoplaced yes)
-		(property "Reference" "#PWR045"
+		(property "Reference" "#PWR034"
 			(at 152.4 127 0)
 			(effects
@@
 			(project "cubesat_rp2040"
 				(path "/5511013b-c214-40ba-8960-f470f52474f8/9f508e75-6f97-47bb-8ac1-2b188f21985e"
-					(reference "#PWR045")
+					(reference "#PWR034")
 					(unit 1)
 				)
@@
 		(dnp no)
 		(fields_autoplaced yes)
-		(property "Reference" "C23"
+		(property "Reference" "C17"
 			(at 232.41 106.6799 0)
 			(effects
@@
 			(project "cubesat_rp2040"
 				(path "/5511013b-c214-40ba-8960-f470f52474f8/9f508e75-6f97-47bb-8ac1-2b188f21985e"
-					(reference "C23")
+					(reference "C17")
 					(unit 1)
 				)
@@
 		(dnp no)
 		(fields_autoplaced yes)
-		(property "Reference" "#PWR043"
+		(property "Reference" "#PWR032"
 			(at 76.2 67.31 0)
 			(effects
@@
 			(project "cubesat_rp2040"
 				(path "/5511013b-c214-40ba-8960-f470f52474f8/9f508e75-6f97-47bb-8ac1-2b188f21985e"
-					(reference "#PWR043")
+					(reference "#PWR032")
 					(unit 1)
 				)
@@
 		(dnp no)
 		(fields_autoplaced yes)
-		(property "Reference" "R21"
+		(property "Reference" "R14"
 			(at 88.9 69.85 90)
 			(effects
@@
 			(project "cubesat_rp2040"
 				(path "/5511013b-c214-40ba-8960-f470f52474f8/9f508e75-6f97-47bb-8ac1-2b188f21985e"
-					(reference "R21")
+					(reference "R14")
 					(unit 1)
 				)
@@
 		(dnp no)
 		(fields_autoplaced yes)
-		(property "Reference" "#PWR044"
+		(property "Reference" "#PWR033"
 			(at 102.87 127 0)
 			(effects
@@
 			(project "cubesat_rp2040"
 				(path "/5511013b-c214-40ba-8960-f470f52474f8/9f508e75-6f97-47bb-8ac1-2b188f21985e"
-					(reference "#PWR044")
+					(reference "#PWR033")
 					(unit 1)
 				)
@@
 		(dnp no)
 		(fields_autoplaced yes)
-		(property "Reference" "C21"
+		(property "Reference" "C15"
 			(at 106.68 100.3299 0)
 			(effects
@@
 			(project "cubesat_rp2040"
 				(path "/5511013b-c214-40ba-8960-f470f52474f8/9f508e75-6f97-47bb-8ac1-2b188f21985e"
-					(reference "C21")
+					(reference "C15")
 					(unit 1)
 				)
@@
 		(dnp no)
 		(fields_autoplaced yes)
-		(property "Reference" "#FLG04"
+		(property "Reference" "#FLG03"
 			(at 152.4 71.755 0)
 			(effects
@@
 			(project "cubesat_rp2040"
 				(path "/5511013b-c214-40ba-8960-f470f52474f8/9f508e75-6f97-47bb-8ac1-2b188f21985e"
-					(reference "#FLG04")
+					(reference "#FLG03")
 					(unit 1)
 				)
@@
 		(dnp no)
 		(fields_autoplaced yes)
-		(property "Reference" "#PWR046"
+		(property "Reference" "#PWR035"
 			(at 228.6 127 0)
 			(effects
@@
 			(project "cubesat_rp2040"
 				(path "/5511013b-c214-40ba-8960-f470f52474f8/9f508e75-6f97-47bb-8ac1-2b188f21985e"
-					(reference "#PWR046")
+					(reference "#PWR035")
 					(unit 1)
 				)
@@
 		(dnp no)
 		(fields_autoplaced yes)
-		(property "Reference" "R22"
+		(property "Reference" "R15"
 			(at 203.2 95.25 90)
 			(effects
@@
 			(project "cubesat_rp2040"
 				(path "/5511013b-c214-40ba-8960-f470f52474f8/9f508e75-6f97-47bb-8ac1-2b188f21985e"
-					(reference "R22")
-					(unit 1)
-				)
+					(reference "R15")
+					(unit 1)
+				)
