File: rp2040.kicad_sch (KiCad schematic)
At the start: 26 parts, among them J501 FTSH-105-01-L-DV-007, U502 RP2040, U503 S25FL128SAGNFM000

Commit message: Another large revision, but we are getting closer
Parts:
- removed R501, R502: 0R, cubesat_rp2040:R_0402_1005Metric, symbol Device:R
- removed R507: 100k, cubesat_rp2040:R_0402_1005Metric, symbol Device:R
- added C30, C76, C78: 100nF, cubesat_rp2040:C_0402_1005Metric, symbol Device:C_Small
- added C75, C79: 10uF, Capacitor_SMD:C_1206_3216Metric, symbol Device:C_Small
- added C77: 1uF, Capacitor_SMD:C_0805_2012Metric, symbol Device:C_Small
- added L4: 15uH, Inductor_SMD:L_1210_3225Metric, symbol Device:L_Small
- added R28, R29, R30: 100kR, cubesat_rp2040:R_0402_1005Metric, symbol Device:R_Small
- added U13: LMR36503MSC3RPERQ1, symbol cubesat_rp2040:LMR36503-Q1
- added U6: 74LVC1G11, Package_TO_SOT_SMD:SOT-563, symbol 74xGxx:74LVC1G11
- C74: renamed from C501; value 100n -> 100nF; LCSC_Part_Number (none) -> C960916; MANUFACTURER (none) -> Samsung Electro-Mechanics; Manufacturer_Part_Number CL31B104KBCNNNC -> CL05B104KB5NNNC
- C81: renamed from C502; value 1u -> 1uF; footprint cubesat_rp2040:C_0402_1005Metric -> Capacitor_SMD:C_0805_2012Metric; LCSC_Part_Number (none) -> C28323; MANUFACTURER (none) -> Samsung Electro-Mechanics; Manufacturer_Part_Number CL31B225KBHNNNE -> CL21B105KBFNNNE
- C82: renamed from C503; value 1u -> 1uF; footprint cubesat_rp2040:C_0402_1005Metric -> Capacitor_SMD:C_0805_2012Metric; LCSC_Part_Number (none) -> C28323; MANUFACTURER (none) -> Samsung Electro-Mechanics; Manufacturer_Part_Number CL31B225KBHNNNE -> CL21B105KBFNNNE
- C83: renamed from C504; value 100n -> 100nF; LCSC_Part_Number (none) -> C960916; MANUFACTURER (none) -> Samsung Electro-Mechanics; Manufacturer_Part_Number CL31B104KBCNNNC -> CL05B104KB5NNNC
- C84: renamed from C505; value 100n -> 100nF; LCSC_Part_Number (none) -> C960916; MANUFACTURER (none) -> Samsung Electro-Mechanics; Manufacturer_Part_Number CL31B104KBCNNNC -> CL05B104KB5NNNC
- C85: renamed from C506; value 100n -> 100nF; LCSC_Part_Number (none) -> C960916; MANUFACTURER (none) -> Samsung Electro-Mechanics; Manufacturer_Part_Number CL31B104KBCNNNC -> CL05B104KB5NNNC
- C86: renamed from C507; value 100n -> 100nF; LCSC_Part_Number (none) -> C960916; MANUFACTURER (none) -> Samsung Electro-Mechanics; Manufacturer_Part_Number CL31B104KBCNNNC -> CL05B104KB5NNNC
- C87: renamed from C508; value 100n -> 100nF; LCSC_Part_Number (none) -> C960916; MANUFACTURER (none) -> Samsung Electro-Mechanics; Manufacturer_Part_Number CL31B104KBCNNNC -> CL05B104KB5NNNC
- C88: renamed from C509; value 100n -> 100nF; LCSC_Part_Number (none) -> C960916; MANUFACTURER (none) -> Samsung Electro-Mechanics; Manufacturer_Part_Number CL31B104KBCNNNC -> CL05B104KB5NNNC
- C89: renamed from C510; value 100n -> 100nF; LCSC_Part_Number (none) -> C960916; MANUFACTURER (none) -> Samsung Electro-Mechanics; Manufacturer_Part_Number CL31B104KBCNNNC -> CL05B104KB5NNNC
- C90: renamed from C511; value 100n -> 100nF; LCSC_Part_Number (none) -> C960916; MANUFACTURER (none) -> Samsung Electro-Mechanics; Manufacturer_Part_Number CL31B104KBCNNNC -> CL05B104KB5NNNC
- C91: renamed from C512; value 100n -> 100nF; LCSC_Part_Number (none) -> C960916; MANUFACTURER (none) -> Samsung Electro-Mechanics; Manufacturer_Part_Number CL31B104KBCNNNC -> CL05B104KB5NNNC
- C92: renamed from C513; value 100n -> 100nF; LCSC_Part_Number (none) -> C960916; MANUFACTURER (none) -> Samsung Electro-Mechanics; Manufacturer_Part_Number CL31B104KBCNNNC -> CL05B104KB5NNNC
- C93: renamed from C514; value 100n -> 100nF; LCSC_Part_Number (none) -> C960916; MANUFACTURER (none) -> Samsung Electro-Mechanics; Manufacturer_Part_Number CL31B104KBCNNNC -> CL05B104KB5NNNC
- C94: renamed from C515; value 100n -> 100nF; LCSC_Part_Number (none) -> C960916; MANUFACTURER (none) -> Samsung Electro-Mechanics; Manufacturer_Part_Number CL31B104KBCNNNC -> CL05B104KB5NNNC
- J7: renamed from J501; value FTSH-105-01-L-DV-007 -> FTSH-105-01-L-DV-007-K; LCSC_Part_Number (none) -> C5296739; Manufacturer_Name (none) -> SAMTEC; Manufacturer_Part_Number (none) -> FTSH-105-01-L-DV-007-K
- R47: renamed from R510; value 1k -> 1kR; LCSC_Part_Number (none) -> C445596; Manufacturer_Name Vishay -> PANASONIC; Manufacturer_Part_Number P-0402E1001FGxx -> ERA2AEB102X
- R48: renamed from R508; symbol Device:R -> Device:R_Small; LCSC_Part_Number (none) -> C25156; Manufacturer_Name Vishay -> UNI-ROYAL(Uniroyal Elec); Manufacturer_Part_Number P-0402E27R0FGxx -> 0402WGJ0270TCE
- R49: renamed from R509; symbol Device:R -> Device:R_Small; LCSC_Part_Number (none) -> C25156; Manufacturer_Name Vishay -> UNI-ROYAL(Uniroyal Elec); Manufacturer_Part_Number P-0402E27R0FGxx -> 0402WGJ0270TCE
- R50: renamed from R505; value 100k -> 100kR; LCSC_Part_Number (none) -> C191569; Manufacturer_Name Vishay -> PANASONIC; Manufacturer_Part_Number P-0402E1003FGxx -> ERA2AED104X
- R51: renamed from R506; value 100k -> 100kR; LCSC_Part_Number (none) -> C191569; Manufacturer_Name Vishay -> PANASONIC; Manufacturer_Part_Number P-0402E1003FGxx -> ERA2AED104X
- U14: renamed from U503; value S25FL128SAGNFM000 -> IS25LP128F; footprint cubesat_rp2040:SON8_S25FL128SAGNFI001_INF -> Package_SO:SOIC-8_5.275x5.275mm_P1.27mm; symbol cubesat_rp2040:S25FL128S -> cubesat_rp2040:IS25LP128F; LCSC_Part_Number (none) -> C1236837; Manufacturer_Name (none) -> ISSI(Integrated Silicon Solution); Manufacturer_Part_Number (none) -> IS25LP128F-JBLA3
- U15: renamed from U502; LCSC_Part_Number (none) -> C2040; Manufacturer_Name (none) -> Raspberry Pi
Connections:
- net GND: now also C30.2, C75.2, C76.2, C77.2, C79.2, U13.9 (GND), U6.2 (GND); no longer U14.9 (EP)
- net RUN: now also U6.4; no longer J7.10 (nSRST)
- net +1V1 renamed +1V1_UNIT
- net +3V3 renamed +3V3_UNIT
- net +3V3_UNIT: now also C30.1, C79.1, L4.2, R28.1, R29.1, R30.1, U13.8 (VOUT/BIAS), U6.5 (VCC)
- net 48M0_CLK renamed 24M0_CLK
- net D+ renamed RP_USB.D+
- net D- renamed RP_USB.D-
- net GPIO10 renamed CAN_B.STB
- net GPIO11 renamed CAN_B.RXD
- net GPIO12 renamed CAN_B.TXD
- net GPIO13 renamed CAN_A.RXD
- net GPIO14 renamed CAN_A.TXD
- net GPIO15 renamed CAN_A.STB
- net GPIO26/ADC0 renamed VOTE_1
- net GPIO27/ADC1 renamed VOTE_2
- net LNM_ENABLE: no longer names the net of U15.40 (GPIO28_ADC2)
- net TESTEN: no longer names the net of U15.19 (TESTEN)
- new net: C77.1, U13.1 (RT), U13.7 (VCC)
- new net BOOT: C78.1, U13.6 (BOOT)
- new net SW: C78.2, L4.1, U13.5 (SW)
- new net VIN: C75.1, C76.1, U13.3 (EN/UVLO), U13.4 (VIN)
- new net ~{PWR_RESET}: R29.2, U13.2 (PGOOD), U6.1
- new net ~{TMR_RESET}: R30.2, U6.6
- new net ~{USR_RESET}: J7.10 (nSRST), R28.2, U6.3
- no-connect marks 31 -> 25
Other:
- added sheet CAN (can.kicad_sch)
- note added: "+3V3 POWER CONVERTER"
- note added: "BOOT FLASH MEMORY"
- note added: "DEBUG CONNECTOR"
- note added: "MCU DECOUPLING CAPS"
- note added: "RESET SIGNAL BUFFER"
- moved on the sheet: C74, C81, C82, C83, C84, C85, C86, C87, C88, C89, C90, C91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

Commit message: Clean up project
Parts:
- renumbered C30 to C80, R28 to R52, R29 to R53, R30 to R54, U6 to U16
Changed lines of the file:
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@@
 		(dnp no)
 		(fields_autoplaced yes)
-		(property "Reference" "R28"
+		(property "Reference" "R52"
 			(at 180.34 34.2899 0)
 			(effects
@@
 		(dnp no)
 		(fields_autoplaced yes)
-		(property "Reference" "C30"
+		(property "Reference" "C80"
 			(at 223.5263 21.59 90)
 			(effects
@@
 		(dnp no)
 		(fields_autoplaced yes)
-		(property "Reference" "#PWR054"
+		(property "Reference" "#PWR092"
 			(at 228.6 36.83 0)
 			(effects
@@
 		(dnp no)
 		(fields_autoplaced yes)
-		(property "Reference" "R30"
+		(property "Reference" "R54"
 			(at 200.66 34.2899 0)
 			(effects
@@
 		(dnp no)
 		(fields_autoplaced yes)
-		(property "Reference" "R29"
+		(property "Reference" "R53"
 			(at 190.5 34.2899 0)
 			(effects
@@
 		(dnp no)
 		(fields_autoplaced yes)
-		(property "Reference" "#PWR053"
+		(property "Reference" "#PWR091"
 			(at 215.9 64.77 0)
 			(effects
@@
 		(dnp no)
 		(fields_autoplaced yes)
-		(property "Reference" "U6"
+		(property "Reference" "U16"
 			(at 228.6 39.4014 0)
 			(effects

Commit message: More work on interfaces
Parts:
- U10: renamed from U13; footprint (none) -> cubesat_rp2040:TI_VQFN-HR_2.1x2.1mm_P0.5mm
- renumbered C74 to C60, C75 to C61, C76 to C62, C77 to C63, C78 to C64, C79 to C65, C80 to C66, C81 to C67, C83 to C68, C84 to C69, C85 to C70, C82 to C71, C86 to C72, C87 to C73, C88 to C74, C89 to C75, C90 to C76, C91 to C77, C92 to C78, C93 to C79, C94 to C80, L4 to L3, R47 to R32, R48 to R33, R49 to R34, R50 to R35, R51 to R36, R52 to R37, R53 to R38, R54 to R39, U14 to U11, U15 to U12, U16 to U13
Connections:
- net CAN_A.STB renamed CAN_A.~{STB}
- net CAN_B.STB renamed CAN_B.~{STB}
- net RUN renamed ~{RESET}
- net VOTE_1 renamed TMR_VOTE_1
- net VOTE_2 renamed TMR_VOTE_2
- net ~{USB_BOOT} renamed FLASH_BOOT/~{USB_BOOT}
Other:
- removed sheet CAN
- moved on the sheet: C65, C68, C69, C70, C71, R32
