File: tmr.kicad_sch (KiCad schematic)
At the start: 9 parts, among them U18 74LVC2G38, U19 74LVC2G38, U20 74LVC2G38

Commit message: More work on interfaces
Parts:
- added C93, C94, C95: 100nF, cubesat_rp2040:C_0402_1005Metric, symbol Device:C
- renumbered D16 to D15, D17 to D16, D18 to D17, R59 to R52, R60 to R53, R61 to R54, U18 to U17, U19 to U18, U20 to U19
Connections:
- net +3V3: now also C93.1, C94.1, C95.1
- net GND: now also C93.2, C94.2, C95.2
- net TMR_RESET_A renamed ~{TMR_RESET_A}
- net TMR_RESET_B renamed ~{TMR_RESET_B}
- net TMR_RESET_C renamed ~{TMR_RESET_C}
Other:
- title: CubeSat RP2040 Board -> TMR RESET VOTING CIRCUIT
